File: PCB/Artificer A1 Board Rev 0.1/processor.kicad_sch (KiCad schematic)
At the start: 8 parts, among them U1 T527M00X0DCH

Commit message: added features
Connections:
- net PCIE0-PERSTN : now reaches U1.A16 (PH11)
- net PCIE0-CLKREQN: now reaches U1.C13 (PH19)
- net PCIE0-WAKEN: now reaches U1.C15 (PH12)
