File: PCB/Artificer A1 Board Rev 0.1/ethernet1.kicad_sch (KiCad schematic)
At the start: 33 parts, among them J3 LPJG0926HENL, J5 PoE, U9 RTL8211F-CG, X3 25MHz

Commit message: finished rough draft of power supply circuitry!
Yay! This one took a while
Connections:
- net +3V3 renamed VCC33-GMAC
Other:
- note added: "VDD_RG (pin 28) determines the signaling level of the RGMII interface. 3.3V is currently selected."
