File: PCB/Artificer A1 Board Rev 0.1/power.kicad_sch (KiCad schematic)
At the start: 181 parts, among them Q1 50P03DF_C21713992, U1 T527M00X0DCH, U13 RT8289GSP, U15 RT8289GSP, U16 ETA8121S2G, U2 AXP323, U4 AXP717B

Commit message: finished rough draft of power supply circuitry!
Yay! This one took a while
Parts:
- removed NT11, NT12, NT13, NT15, NT25, NT26, NT27, NT28, NT31, NT32, NT34, NT35, NT36, NT38, NT41: NetTie_2, symbol Device:NetTie_2
- removed U16: ETA8121S2G, easyeda:SOT-23-6_L2.9-W1.6-P0.95-LS2.9-BL, symbol easyeda:ETA8121S2G
- added C138: 10uF, symbol Device:C_Small
- added C139: 22pF, symbol Device:C_Small
- added C140: 22uF, symbol Device:C_Small
- added C141: 100nF, symbol Device:C_Small
- added L14: 1uH, symbol Device:L
- added NT55, NT56, NT57, NT58, NT59, NT60, NT61, NT62: NetTie_2, symbol Device:NetTie_2
- added R86: 1k, symbol Device:R_Small
- added R87: 100k, symbol Device:R_Small
- added U18: SY8089A1AAC, easyeda:TSOT-23-5_L2.9-W1.6-P0.95-LS2.8-BR, symbol easyeda:SY8089A1AAC
Connections:
- net VDD-DRAM is gone; now on net CPVIN: NT42.2
- net VDD18-LPDDR is gone; now on net VDD18-DRAM: NT24.2
- net +5V: no longer C81.1, C83.1, C84.1, U4.31 (VIN3), U4.32 (VIN2), U4.9 (VIN1)
- net 5V_SYS: now also C81.1, C83.1, C84.1, U4.31 (VIN3), U4.32 (VIN2), U4.9 (VIN1)
- net BLDO1: now also NT23.1
- net BLDO2: now also C141.1, U18.1 (EN); no longer NT23.1
- net BLDO3: now also NT42.1, NT57.1, NT58.1, NT59.1, NT60.1
- net CLDO1: no longer NT33.1
- net CLDO2: now also NT33.1
- net CLDO3: now also NT46.1, NT61.1, NT62.1; no longer NT43.1
- net CLDO4: now also NT43.1
- net DCDC3: now also NT56.1
- net DCDC4: now also NT55.1; no longer NT42.1, NT46.1
- net GND: now also C138.2, C140.2, C141.2, R87.2, U18.2 (GND)
- net PS: now also C138.1, U18.4 (IN)
- net VCC-ADC: now also U1.W7 (VCCADC)
- net VCC-DCXO: now also U1.AD15 (VCCDCXO)
- net VCC-EFUSE: now also U1.R26 (VCCEFUSE)
- net VCC-LVDS0: now also U1.N24 (VCCLVDS0)
- net VCC-LVDS1: now also U1.N9 (VCCLVDS1)
- net VCC-MCSI: now also U1.K13 (VCCMCSI), NT57.2
- net VCC-PC: now also U1.U26 (VCC-PC)
- net VCC-PD: now also NT51.2, U1.L26 (VCC-PD); no longer NT49.2
- net VCC-PE: now also U1.L9 (VCC-PE), NT55.2; no longer NT47.2
- net VCC-PG: now also U1.T9 (VCC-PG)
- net VCC-PI: now also NT49.2, U1.AE16 (VCC-PI); no longer NT51.2
- net VCC-PJ: now also NT48.2, U1.P9 (VCC-PJ)
- net VCC-PK: now also NT47.2, U1.M10 (VCC-PK); no longer NT48.2
- net VCC-PL: now also U1.AE11 (VCC-PL)
- net VCC-PLL: now also U1.AG15 (VCCPLL)
- net VCC-PM: now also U1.AG9 (VCCPM)
- net VCC-RTC: now also U1.AE13 (VCCRTC)
- net VCC18-EDP: now also U1.L22 (VCC18-EDP), NT60.2
- net VCC18-HDMI: now also U1.M21 (VCC18-HDMI), NT58.2
- net VCC18-PCIE: now also U1.J15 (VCC18-PCIE), NT59.2
- net VCC33-USB: now also U1.J19 (VCC33-18-USB), U1.K19 (VCC33-USB), NT61.2; no longer NT52.2
- net VDD-CPUB: now also U1.T19 (VDDCPUB), U1.T21 (VDDCPUB), U1.T22 (VDDCPUB), U1.U18 (VDDCPUB), U1.U19 (VDDCPUB), U1.U21 (VDDCPUB), U1.U22 (VDDCPUB)
- net VDD-CPUL: now also U1.W19 (VDDCPUL), U1.W21 (VDDCPUL), U1.Y19 (VDDCPUL), U1.Y21 (VDDCPUL)
- net VDD-CPUS: now also U1.AC15 (VDDCPUS)
- net VDD-DE: now also U1.N21 (VDDDE), U1.P21 (VDDDE), U1.P22 (VDD-DE)
- net VDD-DNR: now also U1.AA12 (VDDDNR), U1.AA13 (VDDDNR), U1.Y12 (VDDDNR), U1.Y13 (VDDDNR)
- net VDD-GPU: now also U1.T11 (VDDGPU), U1.T13 (VDDGPU), U1.U12 (VDDGPU), U1.U13 (VDDGPU)
- net VDD-SYS: now also U1.R15 (VDDSYS), U1.R17 (VDD-SYS), U1.R18 (VDD-SYS)
- net VDD-VE: now also U1.N13 (VDD-VE), U1.P13 (VDD-VE)
- net VDD09-EDP: now also U1.M22 (VDD09-EDP)
- net VDD09-HDMI: now also U1.L21 (VDD09-HDMI); no longer NT46.2
- net VDD09-PCIE: now also U1.J16 (VDD09-PCIE)
- net VDD09-USB: now also U1.L18 (VDD09-USB)
- net VDD-CPUBFB: now reaches U2.1 (DCDC2)
- net VDD-CPUBFB: now also U1.R22 (VDDCPUBFB), U2.16 (DCDC1)
- net VDD-DNRFB: now reaches U2.4 (DCDC3)
- net VDD-DNRFB: now also U1.AB13 (VDDDNRFB)
- net VDD-CPULFB: now reaches U4.12 (FB1)
- net VDD-CPULFB: now also U1.AA19 (VDDCPULFB)
- net VDD-SYSFB: now reaches U4.34 (FB2)
- net VDD-SYSFB: now also U1.P18 (VDDSYSFB)
- net VDD33: now reaches U1.AC9 (VDD33)
- net VDD33: now also NT62.2
- net VCC33-USB-2: now reaches U1.J18 (VCC33-18-USB-2)
- net VCC33-USB-2: now also NT52.2, U1.L17 (VCC33-USB-2)
- net VCC-IO: now reaches U1.L15 (VCC-IO)
- net VCC-IO: now also NT46.2
- net VCC-GMAC renamed VCC33-GMAC
- net VCC-WIFI renamed VCC33-WIFI
- new net: C139.2, R86.2, R87.1, U18.5 (FB)
- new net: L14.1, U18.3 (LX)
- new net VDD06-DRAM: C139.1, C140.1, L14.2, R86.1
- new net VDD11-DRAM: NT56.2
- no-connect marks 13 -> 16
Other:
- note added: "0.6V feedback"
- note added: "0.6V output"
- note added: "1.8V(OFF)"
- note added: "CPVEE, CPVDD, These pins are used for headphones and negative charge pumps. Probably shouldnt be here"
- note added: "For USB 2.0"
- note added: "The default value of PMIC is 3.3V. needs to be set to 1.8v before used. only use to program efuse"
- note added: "This pin is used for headphones and negative charge pumps. Probably shouldnt be here"
- note added: "VCC33-USB-2 : This is for power to USB 2 periferial (USB 3.0) on the SoC VCC33-USB is for USB0 and USB1 (USB 2.0)"
- note removed: "VDD-CPUBFB"
- note removed: "VDD-CPULFB"
- note removed: "VDD-DNRFB"
- note removed: "VDD-SYSFB"
- moved on the sheet: NT14, NT16, NT17, NT18, NT19, NT20, NT22, NT23, NT29, NT30, NT33, NT37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
