File: PCB/Artificer A1 Board Rev 0.1/power.kicad_sch (KiCad schematic)
At the start: 75 parts, among them U10 AXP717B, U11 AXP323, U9 SY8089A1AAC

Commit message: more routing and decoupling
Parts:
- added R230, R231: 10k, Resistor_SMD:R_0201_0603Metric, symbol Cap:JLCPCB_Res_Custom
- C162, C163: value 100nF -> 10nF; Voltage Rated 16V -> 10V
- R173: value 0Ω -> 1k
- R174: value 0Ω -> 100k; now fitted; now in the parts list
Connections:
- net AP-NMI: now also R231.2
- net AP-RESET: now also R230.2
- net VCC-RTC: now also R230.1, R231.1

Commit message: worked on power pours
Connections:
- net +5V is gone; now on net 5V_SYS: C251.2, C252.2, C267.2, U10.15 (ALDOIN), U10.20 (BLDOIN), U10.25 (CLDOIN)
- net SW_1: now reaches L4.2, U10.45 (SW_1), U10.46 (SW_2)
Other:
- note added: "1.1V"
- note added: "1.5mA"
- note added: "1.7A"
- note added: "1.9A"
- note added: "1.9mA"
- note added: "133.6mA"
- note added: "137.3mA"
- note added: "15.0mA"
- note added: "15.5mA"
- note added: "17.3mA"
- note added: "2.6mA"
- note added: "22.7mA"
- note added: "25.6mA"
- note added: "26.9mA"
- note added: "27.6mA"
- note added: "4.1mA"
- note added: "5.6mA"
- note added: "51.5mA"
- note added: "517mA"
- note added: "536mA"
- note added: "670mA"
- note added: "892.6mA"
- note added: "970mA"
- note added: "In red is max current when under heavy load."
- note added: "Power Supply for 3.3V Analog Part"
- note added: "~28.2mA"

Commit message: finished most of the power
Parts:
- added C354: 22uF, Capacitor_SMD:C_0603_1608Metric, symbol Cap:JLCPCB_Lib_Blank_Cap
Connections:
- net GND: now also C354.1
- net VDD06-DRAM: now also C354.2
Changed lines of the file:
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@@
 	)
 	(junction
+		(at 137.16 113.03)
+		(diameter 0)
+		(color 0 0 0 0)
+	)
+	(junction
 		(at 321.31 30.48)
 		(diameter 0)
@@
 	)
 	(junction
+		(at 140.97 124.46)
+		(diameter 0)
+		(color 0 0 0 0)
+	)
+	(junction
 		(at 252.73 129.54)
 		(diameter 0)
@@
 	(wire
 		(pts
+			(xy 137.16 114.3) (xy 137.16 113.03)
+		)
+		(stroke
+			(width 0)
+			(type default)
+		)
+	)
+	(wire
+		(pts
 			(xy 222.25 66.04) (xy 222.25 62.23)
 		)
@@
 	(wire
 		(pts
-			(xy 127 113.03) (xy 140.97 113.03)
+			(xy 127 113.03) (xy 137.16 113.03)
 		)
 		(stroke
@@
 	(wire
 		(pts
+			(xy 137.16 124.46) (xy 140.97 124.46)
+		)
+		(stroke
+			(width 0)
+			(type default)
+		)
+	)
+	(wire
+		(pts
 			(xy 247.65 46.99) (xy 261.62 46.99)
 		)
@@
 	(wire
 		(pts
+			(xy 137.16 113.03) (xy 140.97 113.03)
+		)
+		(stroke
+			(width 0)
+			(type default)
+		)
+	)
+	(wire
+		(pts
 			(xy 30.48 173.99) (xy 57.15 173.99)
 		)
@@
 	(wire
 		(pts
+			(xy 137.16 121.92) (xy 137.16 124.46)
+		)
+		(stroke
+			(width 0)
+			(type default)
+		)
+	)
+	(wire
+		(pts
 			(xy 162.56 160.02) (xy 162.56 156.21)
 		)
@@
 					(unit 1)
 				)
+			)
+		)
+	)
+	(symbol
+		(lib_id "Cap:JLCPCB_Lib_Blank_Cap")
+		(at 137.16 118.11 180)
+		(unit 1)
+		(body_style 1)
+		(exclude_from_sim no)
+		(in_bom yes)
+		(on_board yes)
+		(in_pos_files yes)
+		(dnp no)
+		(property "Reference" "C354"
+			(at 136.144 114.808 90)
+			(show_name no)
+			(do_not_autoplace no)
+			(effects
+				(font
+					(size 1.27 1.27)
+				)
+			)
+		)
+		(property "Value" "22uF"
+			(at 138.176 119.126 90)
+			(show_name no)
+			(do_not_autoplace no)
+			(effects
+				(font
+					(size 0.8 0.8)
+				)
+				(justify left)
+			)
+		)
+		(property "Footprint" "Capacitor_SMD:C_0603_1608Metric"
+			(at 138.938 118.11 90)
+			(hide yes)
+			(show_name no)
+			(do_not_autoplace no)
+			(effects
+				(font
+					(size 1.27 1.27)
+				)
+			)
+		)
+		(property "Datasheet" ""
+			(at 137.16 118.11 0)
+			(hide yes)
+			(show_name no)
+			(do_not_autoplace no)
+			(effects
+				(font
+					(size 1.27 1.27)
+				)
+			)
+		)
+		(property "Description" ""
+			(at 137.16 118.11 0)
+			(hide yes)
+			(show_name no)
+			(do_not_autoplace no)
+			(effects
+				(font
+					(size 1.27 1.27)
+				)
+			)
+		)
+		(property "Voltage Rated" "6.3V"
+			(at 136.398 119.634 90)
+			(show_name no)
+			(do_not_autoplace no)
+			(effects
+				(font
+					(size 0.8 0.8)
+				)
+				(justify left)
+			)
+		)
+		(pin "1"
+		)
+		(pin "2"
+		)
+		(instances
+			(project "Artificer A1 Board Rev 0.1"
+				(path "/7c37bdb5-94b0-4567-b5ec-a879db855389/ae3e07ef-f034-4788-a69a-5dbad0c7ebc1"
+					(reference "C354")
+					(unit 1)
+				)

Commit message: more power changed mipi csi and dis to aux 3.3V
Changed lines of the file:
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@@
 	)
 	(junction
+		(at 162.56 262.89)
+		(diameter 0)
+		(color 0 0 0 0)
+	)
+	(junction
 		(at 360.68 205.74)
 		(diameter 0)
@@
 	)
 	(junction
+		(at 162.56 266.7)
+		(diameter 0)
+		(color 0 0 0 0)
+	)
+	(junction
 		(at 30.48 196.85)
 		(diameter 0)
@@
 	)
 	(junction
-		(at 30.48 278.13)
-		(diameter 0)
-		(color 0 0 0 0)
-	)
-	(junction
 		(at 327.66 132.08)
 		(diameter 0)
@@
 	)
 	(junction
-		(at 30.48 274.32)
-		(diameter 0)
-		(color 0 0 0 0)
-	)
-	(junction
 		(at 332.74 175.26)
 		(diameter 0)
@@
 	(wire
 		(pts
-			(xy 30.48 281.94) (xy 30.48 278.13)
-		)
-		(stroke
-			(width 0)
-			(type default)
-		)
-	)
-	(wire
-		(pts
 			(xy 93.98 113.03) (xy 96.52 113.03)
 		)
@@
 	(wire
 		(pts
-			(xy 30.48 278.13) (xy 30.48 274.32)
-		)
-		(stroke
-			(width 0)
-			(type default)
-		)
-	)
-	(wire
-		(pts
 			(xy 196.85 50.8) (xy 261.62 50.8)
 		)
@@
 	(wire
 		(pts
+			(xy 162.56 262.89) (xy 162.56 266.7)
+		)
+		(stroke
+			(width 0)
+			(type default)
+		)
+	)
+	(wire
+		(pts
 			(xy 97.79 190.5) (xy 124.46 190.5)
 		)
@@
 	(wire
 		(pts
-			(xy 57.15 278.13) (xy 30.48 278.13)
-		)
-		(stroke
-			(width 0)
-			(type default)
-		)
-	)
-	(wire
-		(pts
 			(xy 388.62 33.02) (xy 388.62 30.48)
 		)
@@
 	(wire
 		(pts
+			(xy 162.56 270.51) (xy 162.56 266.7)
+		)
+		(stroke
+			(width 0)
+			(type default)
+		)
+	)
+	(wire
+		(pts
 			(xy 30.48 173.99) (xy 57.15 173.99)
 		)
@@
 	(wire
 		(pts
-			(xy 57.15 281.94) (xy 30.48 281.94)
-		)
-		(stroke
-			(width 0)
-			(type default)
-		)
-	)
-	(wire
-		(pts
 			(xy 232.41 88.9) (xy 261.62 88.9)
 		)
@@
 	(wire
 		(pts
+			(xy 162.56 266.7) (xy 189.23 266.7)
+		)
+		(stroke
+			(width 0)
+			(type default)
+		)
+	)
+	(wire
+		(pts
 			(xy 30.48 163.83) (xy 30.48 166.37)
 		)
@@
 	(wire
 		(pts
+			(xy 189.23 270.51) (xy 162.56 270.51)
+		)
+		(stroke
+			(width 0)
+			(type default)
+		)
+	)
+	(wire
+		(pts
 			(xy 341.63 142.24) (xy 337.82 142.24)
 		)
@@
 	(symbol
 		(lib_id "power:+5V")
-		(at 57.15 281.94 0)
+		(at 189.23 266.7 0)
 		(unit 1)
 		(body_style 1)
@@
 		(dnp no)
 		(property "Reference" "#PWR0162"
-			(at 57.15 285.75 0)
+			(at 189.23 270.51 0)
 			(hide yes)
 			(show_name no)
@@
 		)
 		(property "Value" "VCC3V3-CSI"
-			(at 49.784 280.416 0)
+			(at 181.864 265.176 0)
 			(show_name no)
 			(do_not_autoplace no)
@@
 		)
 		(property "Footprint" ""
-			(at 57.15 281.94 0)
+			(at 189.23 266.7 0)
 			(hide yes)
 			(show_name no)
@@
 		)
 		(property "Datasheet" ""
-			(at 57.15 281.94 0)
+			(at 189.23 266.7 0)
 			(hide yes)
 			(show_name no)
@@
 		)
 		(property "Description" "Power symbol creates a global label with name \"+5V\""
-			(at 57.15 281.94 0)
+			(at 189.23 266.7 0)
 			(hide yes)
 			(show_name no)
@@
 	(symbol
 		(lib_id "power:+5V")
-		(at 57.15 278.13 0)
+		(at 189.23 270.51 0)
 		(unit 1)
 		(body_style 1)
@@
 		(dnp no)
 		(property "Reference" "#PWR0161"
-			(at 57.15 281.94 0)
+			(at 189.23 274.32 0)
 			(hide yes)
 			(show_name no)
@@
 		)
 		(property "Value" "VCC-LCD"
-			(at 49.784 276.606 0)
+			(at 181.864 268.986 0)
 			(show_name no)
 			(do_not_autoplace no)
@@
 		)
 		(property "Footprint" ""
-			(at 57.15 278.13 0)
+			(at 189.23 270.51 0)
 			(hide yes)
 			(show_name no)
@@
 		)
 		(property "Datasheet" ""
-			(at 57.15 278.13 0)
+			(at 189.23 270.51 0)
 			(hide yes)
 			(show_name no)
@@
 		)
 		(property "Description" "Power symbol creates a global label with name \"+5V\""
-			(at 57.15 278.13 0)
+			(at 189.23 270.51 0)
 			(hide yes)
 			(show_name no)
