File: PCB/Artificer A1 Board Rev 0.1/Artificer A1 Board Rev 0.1.kicad_sch (KiCad schematic)
At the start: 7 parts, among them M1 Fan&Heatsink_30x30mm

Commit message: finsihed more routing
Parts:
- removed M1: Fan&Heatsink_30x30mm, custom footprints:custom_heatsink&fan, symbol Fan:Fan&Heatsink_30x30mm
- added M1: Fan&Heatsink_40x40mm, custom footprints:custom_heatsink&fan_40x40mm, symbol Fan:Fan&Heatsink_40x40mm
Connections:
- new net GND: M1.1 (MP), M1.2 (MP), M1.3 (MP), M1.4 (MP)
Other:
- sheet T527 ports: added {PMIC-TWI}; removed none
- sheet power ports: added {PMIC-TWI}; removed none
- sheet power input ports: added {USB_DRD}; removed none
- sheet usb ports: added none; removed {USB_DRD}
