File: PCB/Artificer A1 Board Rev 0.1/Artificer A1 Board Rev 0.1.kicad_sch (KiCad schematic)
At the start: 7 parts, among them M1 Fan&Heatsink_40x40mm

Commit message: more routing and decoupling
Other:
- sheet T527 ports: added {GPIO}; removed none
- sheet gpio ports: added {GPIO}; removed none
Changed lines of the file:
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@@
+	(bus
+		(pts
+			(xy 72.39 95.25) (xy 80.01 95.25)
+		)
+		(stroke
+			(width 0)
+			(type default)
+		)
+	)
 	(bus
 		(pts
@@
 			)
 		)
+		(pin "{GPIO}" bidirectional
+			(at 72.39 95.25 0)
+			(effects
+				(font
+					(size 1.27 1.27)
+				)
+				(justify right)
+			)
+		)
 		(instances
 			(project "Artificer A1 Board Rev 0.1"
@@
 			)
 		)
+		(pin "{GPIO}" bidirectional
+			(at 80.01 95.25 180)
+			(effects
+				(font
+					(size 1.27 1.27)
+				)
+				(justify left)
+			)
+		)
