File: PCB/Artificer A1 Board Rev 0.1/Artificer A1 Board Rev 0.1.kicad_pcb (KiCad board)
At the start: 2 copper layers, 0 parts

Commit message: placed all components
Parts:
- added C1: 10uF, PCM_JLCPCB:C_0805, B.Cu at (130.3, 133.7)
- added C13: 1uF, PCM_JLCPCB:C_0402, F.Cu at (145.3, 127.3)
- added C133: 100nF, Capacitor_SMD:C_0201_0603Metric, F.Cu at (82.6, 71.6)
- added C134: 100nF, Capacitor_SMD:C_0201_0603Metric, F.Cu at (136.8, 89.1)
- added C135: 100nF, Capacitor_SMD:C_0201_0603Metric, F.Cu at (136.8, 89.8)
- added C136: 100nF, Capacitor_SMD:C_0201_0603Metric, F.Cu at (136.8, 90.7)
- added C137: 100nF, Capacitor_SMD:C_0201_0603Metric, F.Cu at (136.8, 91.4)
- added C138: 100nF, Capacitor_SMD:C_0201_0603Metric, F.Cu at (136.8, 92.8)
- added C139: 100nF, Capacitor_SMD:C_0201_0603Metric, F.Cu at (136.8, 93.5)
- added C14: 10uF, PCM_JLCPCB:C_0805, B.Cu at (139.4, 133.8)
- added C140: 100nF, Capacitor_SMD:C_0201_0603Metric, F.Cu at (136.8, 94.3)
- added C141: 100nF, Capacitor_SMD:C_0201_0603Metric, F.Cu at (136.8, 95.1)
- added C142: 100nF, Capacitor_SMD:C_0201_0603Metric, F.Cu at (140.9, 100.8)
- added C143: 100nF, Capacitor_SMD:C_0201_0603Metric, F.Cu at (140.9, 100.0)
- added C15: 10uF, PCM_JLCPCB:C_0805, B.Cu at (139.3, 120.5)
- added C151: 100nF, Capacitor_SMD:C_0201_0603Metric, F.Cu at (73.6, 73.9)
- added C154: 100nF, Capacitor_SMD:C_0201_0603Metric, F.Cu at (65.9, 71.2)
- added C158: 100nF, Capacitor_SMD:C_0201_0603Metric, F.Cu at (78.7, 80.5)
- added C159: 100nF, Capacitor_SMD:C_0201_0603Metric, F.Cu at (119.2, 101.4)
- added C16: 100nF, PCM_JLCPCB:C_0402, F.Cu at (135.8, 130.5)
- added C160: 100nF, Capacitor_SMD:C_0201_0603Metric, F.Cu at (82.8, 80.1)
- added C161: 100nF, Capacitor_SMD:C_0201_0603Metric, F.Cu at (56.9, 73.6)
- added C162: 100nF, Capacitor_SMD:C_0201_0603Metric, F.Cu at (131.0, 110.1)
- added C163: 100nF, Capacitor_SMD:C_0201_0603Metric, F.Cu at (122.5, 110.7)
- added C164: 100nF, Capacitor_SMD:C_0201_0603Metric, F.Cu at (143.7, 71.0)
- added C165: 100nF, Capacitor_SMD:C_0201_0603Metric, F.Cu at (119.2, 96.5)
- added C166: 2.2uF, Capacitor_SMD:C_0201_0603Metric, F.Cu at (82.8, 80.9)
- added C167: 100nF, Capacitor_SMD:C_0201_0603Metric, F.Cu at (58.6, 108.7)
- added C168: 100nF, Capacitor_SMD:C_0201_0603Metric, F.Cu at (62.0, 80.1)
- added C169: 2.2uF, Capacitor_SMD:C_0201_0603Metric, F.Cu at (66.1, 80.5)
- added C17: 100nF, PCM_JLCPCB:C_0402, F.Cu at (135.6, 117.4)
- added C170: 100nF, Capacitor_SMD:C_0201_0603Metric, F.Cu at (66.1, 79.8)
- added C171: 100nF, Capacitor_SMD:C_0201_0603Metric, B.Cu at (107.0, 70.1)
- added C172: 100nF, Capacitor_SMD:C_0201_0603Metric, B.Cu at (111.0, 77.2)
- added C176: 100nF, Capacitor_SMD:C_0201_0603Metric, B.Cu at (97.4, 88.3)
- added C177: 100nF, Capacitor_SMD:C_0201_0603Metric, B.Cu at (106.0, 77.4)
- added C178: 100nF, Capacitor_SMD:C_0201_0603Metric, B.Cu at (111.1, 71.6)
- added C179: 22uF, Capacitor_SMD:C_0603_1608Metric, B.Cu at (111.0, 70.4)
- added C180: 22uF, Capacitor_SMD:C_0603_1608Metric, B.Cu at (111.0, 78.3)
- added C181: 100nF, Capacitor_SMD:C_0201_0603Metric, F.Cu at (118.0, 126.2)
- added C182: 22pF, Capacitor_SMD:C_0201_0603Metric, F.Cu at (116.3, 125.2)
- added C183: 100nF, Capacitor_SMD:C_0201_0603Metric, F.Cu at (58.6, 109.5)
- added C184: 100nF, Capacitor_SMD:C_0201_0603Metric, F.Cu at (58.6, 110.3)
- added C185: 100nF, Capacitor_SMD:C_0201_0603Metric, F.Cu at (58.6, 108.0)
- added C186: 100nF, Capacitor_SMD:C_0201_0603Metric, F.Cu at (127.1, 73.6)
- added C187: 100nF, Capacitor_SMD:C_0201_0603Metric, F.Cu at (116.4, 102.2)
- added C188: 22pF, Capacitor_SMD:C_0201_0603Metric, F.Cu at (142.6, 127.7)
- added C189: 100nF, Capacitor_SMD:C_0201_0603Metric, F.Cu at (60.0, 121.2)
- added C190: 1uF, Capacitor_SMD:C_0201_0603Metric, F.Cu at (60.0, 122.0)
- added C191: 100nF, Capacitor_SMD:C_0201_0603Metric, F.Cu at (71.8, 126.4)
- added C192: 1uF, Capacitor_SMD:C_0201_0603Metric, F.Cu at (72.5, 126.4)
- added C193: 100nF, Capacitor_SMD:C_0201_0603Metric, F.Cu at (57.1, 95.6)
- added C194: 1uF, Capacitor_SMD:C_0201_0603Metric, F.Cu at (57.1, 96.3)
- added C195: 3.3nF, Capacitor_SMD:C_0201_0603Metric, F.Cu at (142.0, 130.9)
- added C196: 47pF, Capacitor_SMD:C_0201_0603Metric, F.Cu at (142.7, 129.4)
- added C197: 3.3nF, Capacitor_SMD:C_0201_0603Metric, F.Cu at (141.8, 117.6)
- added C198: 100nF, Capacitor_SMD:C_0201_0603Metric, B.Cu at (112.5, 114.4)
- added C199: 100nF, Capacitor_SMD:C_0201_0603Metric, B.Cu at (102.7, 114.4)
- added C2: 100nF, PCM_JLCPCB:C_0402, F.Cu at (126.5, 130.5)
- added C200: 100nF, Capacitor_SMD:C_0201_0603Metric, B.Cu at (101.3, 117.6)
- added C201: 100nF, Capacitor_SMD:C_0201_0603Metric, B.Cu at (101.2, 120.0)
- added C202: 100nF, Capacitor_SMD:C_0201_0603Metric, B.Cu at (114.4, 121.6)
- added C203: 100nF, Capacitor_SMD:C_0201_0603Metric, B.Cu at (113.8, 120.0)
- added C204: 47pF, Capacitor_SMD:C_0201_0603Metric, F.Cu at (142.6, 116.2)
- added C205: 22pF, Capacitor_SMD:C_0201_0603Metric, F.Cu at (142.4, 114.2)
- added C206: 100nF, Capacitor_SMD:C_0201_0603Metric, B.Cu at (114.4, 116.0)
- added C207: 100nF, Capacitor_SMD:C_0201_0603Metric, F.Cu at (136.8, 96.8)
- added C208: 100nF, Capacitor_SMD:C_0201_0603Metric, F.Cu at (136.8, 97.6)
- added C209: 2.2uF, Capacitor_SMD:C_0201_0603Metric, F.Cu at (79.5, 80.5)
- added C210: 2.2uF, Capacitor_SMD:C_0201_0603Metric, F.Cu at (62.8, 80.1)
- added C211: 100nF, Capacitor_SMD:C_0201_0603Metric, F.Cu at (73.2, 79.2)
- added C212: 100nF, Capacitor_SMD:C_0201_0603Metric, F.Cu at (56.5, 78.9)
- added C213: 100nF, Capacitor_SMD:C_0201_0603Metric, F.Cu at (73.2, 78.5)
- added C214: 100nF, Capacitor_SMD:C_0201_0603Metric, F.Cu at (56.5, 78.1)
- added C215: 6pF, Capacitor_SMD:C_0201_0603Metric, F.Cu at (82.2, 75.6)
- added C216: 6pF, Capacitor_SMD:C_0201_0603Metric, F.Cu at (65.5, 75.3)
- added C217: 6pF, Capacitor_SMD:C_0201_0603Metric, F.Cu at (82.2, 73.7)
- added C218: 6pF, Capacitor_SMD:C_0201_0603Metric, F.Cu at (65.5, 73.4)
- added C219: 1uF, Capacitor_SMD:C_0201_0603Metric, F.Cu at (151.9, 115.9)
- added C220: 1uF, Capacitor_SMD:C_0201_0603Metric, F.Cu at (152.9, 115.9)
- added C221: 2.2uF, Capacitor_SMD:C_0201_0603Metric, F.Cu at (125.5, 117.4)
- added C222: 2.2uF, Capacitor_SMD:C_0201_0603Metric, F.Cu at (126.2, 117.4)
- added C223: 2.2uF, Capacitor_SMD:C_0201_0603Metric, F.Cu at (127.0, 117.4)
- added C224: 2.2uF, Capacitor_SMD:C_0201_0603Metric, F.Cu at (127.7, 117.4)
- added C225: 2.2uF, Capacitor_SMD:C_0201_0603Metric, F.Cu at (131.0, 115.2)
- added C226: 2.2uF, Capacitor_SMD:C_0201_0603Metric, F.Cu at (130.0, 117.4)
- added C227: 2.2uF, Capacitor_SMD:C_0201_0603Metric, F.Cu at (129.2, 117.4)
- added C228: 2.2uF, Capacitor_SMD:C_0201_0603Metric, F.Cu at (128.5, 117.4)
- added C229: 2.2uF, Capacitor_SMD:C_0201_0603Metric, F.Cu at (122.4, 114.7)
- added C230: 2.2uF, Capacitor_SMD:C_0201_0603Metric, F.Cu at (131.0, 114.5)
- added C231: 1uF, Capacitor_SMD:C_0201_0603Metric, F.Cu at (122.4, 113.1)
- added C232: 1uF, Capacitor_SMD:C_0201_0603Metric, F.Cu at (131.0, 112.7)
- added C233: 22uF, Capacitor_SMD:C_0603_1608Metric, F.Cu at (119.4, 116.7)
- added C234: 22uF, Capacitor_SMD:C_0603_1608Metric, F.Cu at (120.9, 116.7)
- added C235: 22uF, Capacitor_SMD:C_0603_1608Metric, F.Cu at (134.3, 109.0)
- added C236: 22uF, Capacitor_SMD:C_0603_1608Metric, F.Cu at (132.8, 109.0)
- added C237: 22uF, Capacitor_SMD:C_0603_1608Metric, F.Cu at (134.2, 117.2)
- added C238: 22uF, Capacitor_SMD:C_0603_1608Metric, F.Cu at (132.7, 117.2)
- added C239: 22uF, Capacitor_SMD:C_0603_1608Metric, F.Cu at (129.9, 107.3)
- added C240: 22uF, Capacitor_SMD:C_0603_1608Metric, F.Cu at (129.9, 105.8)
- added C241: 2.2uF, Capacitor_SMD:C_0201_0603Metric, F.Cu at (115.6, 103.6)
- added C242: 22uF, Capacitor_SMD:C_0603_1608Metric, F.Cu at (125.1, 106.9)
- added C243: 10uF, Capacitor_SMD:C_0402_1005Metric, F.Cu at (123.8, 107.5)
- added C244: 10uF, Capacitor_SMD:C_0402_1005Metric, F.Cu at (122.9, 107.5)
- added C245: 10uF, Capacitor_SMD:C_0402_1005Metric, F.Cu at (121.9, 107.5)
- added C246: 10uF, Capacitor_SMD:C_0402_1005Metric, F.Cu at (120.9, 107.5)
- added C247: 1uF, Capacitor_SMD:C_0201_0603Metric, F.Cu at (131.0, 113.5)
- added C248: 1uF, Capacitor_SMD:C_0201_0603Metric, F.Cu at (122.4, 112.3)
- added C249: 1uF, Capacitor_SMD:C_0201_0603Metric, F.Cu at (131.0, 110.9)
- added C25: 22uF, PCM_JLCPCB:C_0805, F.Cu at (142.3, 125.3)
- added C250: 1uF, Capacitor_SMD:C_0201_0603Metric, F.Cu at (131.0, 111.6)
- added C251: 1uF, Capacitor_SMD:C_0201_0603Metric, B.Cu at (126.6, 116.0)
- added C252: 1uF, Capacitor_SMD:C_0201_0603Metric, B.Cu at (124.6, 116.0)
- added C253: 2.2uF, Capacitor_SMD:C_0201_0603Metric, F.Cu at (123.2, 117.4)
- added C254: 2.2uF, Capacitor_SMD:C_0201_0603Metric, F.Cu at (124.0, 117.4)
- added C255: 2.2uF, Capacitor_SMD:C_0201_0603Metric, F.Cu at (124.7, 117.4)
- added C256: 10uF, Capacitor_SMD:C_0402_1005Metric, F.Cu at (127.1, 74.5)
- added C257: 1uF, Capacitor_SMD:C_0201_0603Metric, F.Cu at (127.0, 75.5)
- added C258: 1uF, Capacitor_SMD:C_0402_1005Metric, F.Cu at (129.6, 73.0)
- added C259: 4pF, Capacitor_SMD:C_0201_0603Metric, F.Cu at (126.5, 68.3)
- added C260: 4pF, Capacitor_SMD:C_0201_0603Metric, F.Cu at (121.1, 68.3)
- added C261: 22uF, Capacitor_SMD:C_0603_1608Metric, B.Cu at (118.7, 67.3)
- added C262: 22uF, Capacitor_SMD:C_0603_1608Metric, B.Cu at (117.2, 67.3)
- added C263: 22uF, Capacitor_SMD:C_0603_1608Metric, B.Cu at (98.9, 67.2)
- added C264: 22uF, Capacitor_SMD:C_0603_1608Metric, B.Cu at (100.4, 67.2)
- added C265: 22uF, Capacitor_SMD:C_0603_1608Metric, B.Cu at (137.4, 66.0)
- added C266: 22uF, Capacitor_SMD:C_0603_1608Metric, B.Cu at (135.9, 66.0)
- added C267: 1uF, Capacitor_SMD:C_0201_0603Metric, B.Cu at (128.6, 116.2)
- added C268: 22uF, Capacitor_SMD:C_0603_1608Metric, F.Cu at (114.8, 127.4)
- added C269: 10uF, Capacitor_SMD:C_0402_1005Metric, F.Cu at (123.0, 127.4)
- added C27: 22uF, PCM_JLCPCB:C_0805, F.Cu at (142.3, 123.3)
- added C270: 2.2uF, Capacitor_SMD:C_0201_0603Metric, F.Cu at (117.9, 103.6)
- added C271: 2.2uF, Capacitor_SMD:C_0201_0603Metric, F.Cu at (119.4, 107.4)
- added C272: 1uF, Capacitor_SMD:C_0201_0603Metric, F.Cu at (119.4, 106.0)
- added C273: 10uF, Capacitor_SMD:C_0402_1005Metric, F.Cu at (115.4, 110.8)
- added C274: 10uF, Capacitor_SMD:C_0402_1005Metric, F.Cu at (116.4, 110.8)
- added C275: 10uF, Capacitor_SMD:C_0402_1005Metric, F.Cu at (111.0, 110.2)
- added C276: 10uF, Capacitor_SMD:C_0402_1005Metric, F.Cu at (111.0, 109.2)
- added C277: 10uF, Capacitor_SMD:C_0402_1005Metric, F.Cu at (111.0, 103.3)
- added C278: 10uF, Capacitor_SMD:C_0402_1005Metric, F.Cu at (111.0, 102.4)
- added C279: 4.7uF, Capacitor_SMD:C_0402_1005Metric, F.Cu at (114.2, 105.5)
- added C280: 4.7uF, Capacitor_SMD:C_0402_1005Metric, F.Cu at (114.2, 108.2)
- added C281: 4.7uF, Capacitor_SMD:C_0402_1005Metric, F.Cu at (115.9, 109.2)
- added C282: 1uF, Capacitor_SMD:C_0201_0603Metric, B.Cu at (105.9, 120.0)
- added C283: 1uF, Capacitor_SMD:C_0201_0603Metric, B.Cu at (110.5, 120.0)
- added C284: 1uF, Capacitor_SMD:C_0201_0603Metric, F.Cu at (110.5, 124.3)
- added C285: 1uF, Capacitor_SMD:C_0201_0603Metric, F.Cu at (103.6, 124.4)
- added C286: 100nF, Capacitor_SMD:C_0201_0603Metric, B.Cu at (111.1, 116.0)
- added C287: 2.2uF, Capacitor_SMD:C_0201_0603Metric, B.Cu at (112.4, 117.6)
- added C288: 2.2uF, Capacitor_SMD:C_0201_0603Metric, B.Cu at (113.8, 117.6)
- added C289: 3.3nF, Capacitor_SMD:C_0201_0603Metric, F.Cu at (132.7, 130.6)
- added C290: 47pF, Capacitor_SMD:C_0201_0603Metric, F.Cu at (133.5, 129.1)
- added C291: 22pF, Capacitor_SMD:C_0201_0603Metric, F.Cu at (133.3, 127.4)
- added C292: 22uF, Capacitor_SMD:C_0603_1608Metric, F.Cu at (142.2, 112.5)
- added C293: 22uF, Capacitor_SMD:C_0603_1608Metric, F.Cu at (142.2, 111.0)
- added C294: 22uF, Capacitor_SMD:C_0603_1608Metric, F.Cu at (142.2, 109.5)
- added C295: 22uF, Capacitor_SMD:C_0603_1608Metric, F.Cu at (132.5, 125.6)
- added C296: 22uF, Capacitor_SMD:C_0603_1608Metric, F.Cu at (132.5, 124.2)
- added C297: 22uF, Capacitor_SMD:C_0603_1608Metric, F.Cu at (132.5, 122.7)
- added C298: 6.2pF, Capacitor_SMD:C_0201_0603Metric, F.Cu at (51.1, 120.7)
- added C299: 0.4pF, Capacitor_SMD:C_0201_0603Metric, F.Cu at (51.1, 114.8)
- added C3: 1uF, PCM_JLCPCB:C_0402, F.Cu at (150.9, 116.1)
- added C300: 100nF, Capacitor_SMD:C_0201_0603Metric, F.Cu at (58.1, 93.8)
- added C301: 100nF, Capacitor_SMD:C_0201_0603Metric, F.Cu at (100.7, 88.4)
- added C302: 22uF, Capacitor_SMD:C_0603_1608Metric, B.Cu at (107.0, 71.2)
- added C303: 22uF, Capacitor_SMD:C_0603_1608Metric, B.Cu at (106.0, 78.6)
- added C85: 100nF, Capacitor_SMD:C_0201_0603Metric, F.Cu at (96.0, 92.8)
- added C86: 100nF, Capacitor_SMD:C_0201_0603Metric, F.Cu at (96.7, 92.8)
- added C87: 100nF, Capacitor_SMD:C_0201_0603Metric, F.Cu at (98.4, 92.8)
- added C88: 100nF, Capacitor_SMD:C_0201_0603Metric, F.Cu at (97.7, 92.8)
- added C9: 100nF, PCM_JLCPCB:C_0402, F.Cu at (144.6, 110.7)
- added Card1: TF-110, easyeda:TF-SMD_TF-110, B.Cu at (59.1, 95.8)
- added D1: ESDA25P35-1U1M-ES, easyeda:DFN1610-2L_L1.6-W1.0-P1.10-RD, F.Cu at (146.7, 127.5)
- added D10: RClamp0524PATCT, easyeda:SLP2510P8_L2.5-W1.0-P0.50-BL, F.Cu at (116.6, 67.7)
- added D11: RClamp0524PATCT, easyeda:SLP2510P8_L2.5-W1.0-P0.50-BL, F.Cu at (99.5, 67.5)
- added D12: LESD5D5.0CT1G_C5199850, easyeda:SOD-523_L1.2-W0.8-LS1.6-BI, F.Cu at (146.3, 124.8)
- added D13: RClamp0524PATCT, easyeda:SLP2510P8_L2.5-W1.0-P0.50-BL, F.Cu at (146.3, 122.7)
- added D14: LESD5D5.0CT1G_C5199850, easyeda:SOD-523_L1.2-W0.8-LS1.6-BI, F.Cu at (146.3, 120.7)
- added D15: B5819WT_C7502714, easyeda:SOD-523_L1.2-W0.8-LS1.6-RD, F.Cu at (149.8, 116.2)
- added D3: ESDA25P35-1U1M-ES, easyeda:DFN1610-2L_L1.6-W1.0-P1.10-RD, F.Cu at (145.2, 107.9)
- added D4: RClamp0524PATCT, easyeda:SLP2510P8_L2.5-W1.0-P0.50-BL, F.Cu at (142.4, 61.9)
- added D5: RClamp0524PATCT, easyeda:SLP2510P8_L2.5-W1.0-P0.50-BL, F.Cu at (142.4, 65.0)
- added D6: RClamp0524PATCT, easyeda:SLP2510P8_L2.5-W1.0-P0.50-BL, F.Cu at (142.4, 68.0)
- added D7: RClamp0524PATCT, easyeda:SLP2510P8_L2.5-W1.0-P0.50-BL, F.Cu at (138.9, 90.5)
- added D8: RClamp0524PATCT, easyeda:SLP2510P8_L2.5-W1.0-P0.50-BL, F.Cu at (139.1, 93.9)
- added D9: RClamp0524PATCT, easyeda:SLP2510P8_L2.5-W1.0-P0.50-BL, F.Cu at (139.2, 97.7)
- added DP1: CAR06-201EN5F, easyeda:DP-SMD_CAR06-201EN5F, F.Cu at (146.7, 94.8)
- added FPC1: 0.5K-A-22PB, easyeda:FPC-SMD_22P-P1.00_0.5K-A-22PB, F.Cu at (124.8, 94.4)
- added FPC2: 0.5K-A-22PB, easyeda:FPC-SMD_22P-P1.00_0.5K-A-22PB, F.Cu at (124.8, 99.0)
- added H1: MountingHole, custom footprints:NP-mounting-hole, F.Cu at (53.5, 82.5)
- added H2: MountingHole, custom footprints:NP-mounting-hole, F.Cu at (53.5, 131.5)
- added H3: MountingHole, custom footprints:NP-mounting-hole, F.Cu at (111.5, 82.5)
- added H4: MountingHole, custom footprints:NP-mounting-hole, F.Cu at (111.5, 131.5)
- added H5: MountingHole, custom footprints:NP-mounting-hole, F.Cu at (151.5, 53.5)
- added H6: MountingHole, custom footprints:NP-mounting-hole, F.Cu at (151.5, 131.5)
- added HDMI1: HD-A-05H9191N, easyeda:HDMI-SMD_HD-A-05H9192N, F.Cu at (148.8, 65.0)
- added J1: Conn_02x20_Odd_Even, Connector_PinHeader_2.54mm:PinHeader_2x20_P2.54mm_Vertical, F.Cu at (58.4, 132.8)
- added J2: Conn_01x02, Connector_PinHeader_1.27mm:PinHeader_1x02_P1.27mm_Vertical, F.Cu at (103.0, 88.5)
- added JP1: U.FL-R-SMT-1(80), easyeda:RF-SMD_FRF05002-JSS103M, F.Cu at (58.0, 113.8)
- added L10: APH252012C1R0MP01, easyeda:IND-SMD_APH252012C3R3MP01, F.Cu at (118.1, 110.5)
- added L11: APH141208C2R2MP01, easyeda:IND-SMD_L1.4-W1.2_AOTA-B141206SR47MT, F.Cu at (81.1, 80.1)
- added L12: APH141208C2R2MP01, easyeda:IND-SMD_L1.4-W1.2_AOTA-B141206SR47MT, F.Cu at (64.4, 79.8)
- added L13: ANT162442DT-2001A2, easyeda:ANT-SMD_6P-L1.6-W0.8-L, F.Cu at (51.1, 116.8)
- added L14: MLG1005S1N3BT000, easyeda:L0402, F.Cu at (55.8, 117.4)
- added L15: 10uH MTQH404030S100MBT, easyeda:IND-SMD_L4.1-W4.1_MTQH404030S, F.Cu at (138.3, 124.3)
- added L16: 3.3uH MTQH404020S3R3MBT, easyeda:IND-SMD_L4.1-W4.1_MTQH404020S, F.Cu at (128.6, 124.2)
- added L2: 3.3uH MTQH404020S3R3MBT, easyeda:IND-SMD_L4.1-W4.1_MTQH404020S, F.Cu at (138.3, 111.0)
- added L3: APH252012C1R0MP01, easyeda:IND-SMD_APH252012C3R3MP01, F.Cu at (117.0, 128.3)
- added L4: APH252012C1R0MP01, easyeda:IND-SMD_APH252012C3R3MP01, F.Cu at (127.0, 107.0)
- added L5: APH252012C1R0MP01, easyeda:IND-SMD_APH252012C3R3MP01, F.Cu at (120.2, 113.9)
- added L6: APH252012C1R0MP01, easyeda:IND-SMD_APH252012C3R3MP01, F.Cu at (133.4, 111.8)
- added L7: APH252012C1R0MP01, easyeda:IND-SMD_APH252012C3R3MP01, F.Cu at (133.4, 114.4)
- added L8: APH252012C1R0MP01, easyeda:IND-SMD_APH252012C3R3MP01, F.Cu at (111.3, 105.1)
- added L9: APH252012C1R0MP01, easyeda:IND-SMD_APH252012C3R3MP01, F.Cu at (111.4, 107.5)
- added PS1: CPUSLDO, TestPoint:TestPoint_Pad_D1.0mm, F.Cu at (123.2, 105.3)
- added Q1: AON3419-TP, easyeda:DFN-8_L3.0-W3.0-P0.65-BL, F.Cu at (146.7, 115.0)
- added Q2: AON3419-TP, easyeda:DFN-8_L3.0-W3.0-P0.65-BL, F.Cu at (146.7, 110.7)
- added Q3: AO3401A, PCM_JLCPCB:Q_SOT-23, B.Cu at (143.3, 132.1)
- added Q4: 2SK3018, easyeda:SOT-23-3_L2.9-W1.4-P1.90-LS2.6-BR, F.Cu at (56.7, 92.5)
- added Q6: AO3401A, Package_TO_SOT_SMD:SOT-23, F.Cu at (141.2, 71.9)
- added Q7: AO3401A, Package_TO_SOT_SMD:SOT-23, F.Cu at (138.7, 102.7)
- added R107: 10k, Resistor_SMD:R_0201_0603Metric, F.Cu at (136.8, 96.1)
- added R108: 10k, Resistor_SMD:R_0201_0603Metric, F.Cu at (136.8, 98.3)
- added R109: 100k, Resistor_SMD:R_0201_0603Metric, F.Cu at (137.0, 99.7)
- added R110: 100k, Resistor_SMD:R_0201_0603Metric, F.Cu at (143.7, 72.5)
- added R111: 100k, Resistor_SMD:R_0201_0603Metric, F.Cu at (141.3, 103.4)
- added R112: 2.49k, Resistor_SMD:R_0201_0603Metric, F.Cu at (82.6, 72.3)
- added R113: 2.49k, Resistor_SMD:R_0201_0603Metric, F.Cu at (65.9, 72.0)
- added R114: 4.7k, Resistor_SMD:R_0201_0603Metric, F.Cu at (74.2, 80.5)
- added R115: 4.7k, Resistor_SMD:R_0201_0603Metric, F.Cu at (57.5, 80.1)
- added R116: 4.7k, Resistor_SMD:R_0201_0603Metric, F.Cu at (78.0, 80.5)
- added R117: 4.7k, Resistor_SMD:R_0201_0603Metric, F.Cu at (61.3, 80.1)
- added R118: 4.7k, Resistor_SMD:R_0201_0603Metric, F.Cu at (77.2, 80.5)
- added R119: 4.7k, Resistor_SMD:R_0201_0603Metric, F.Cu at (60.5, 80.1)
- added R120: 4.7k, Resistor_SMD:R_0201_0603Metric, F.Cu at (83.1, 78.4)
- added R121: 4.7k, Resistor_SMD:R_0201_0603Metric, F.Cu at (66.4, 78.1)
- added R122: 4.7k, Resistor_SMD:R_0201_0603Metric, F.Cu at (83.1, 77.7)
- added R123: 4.7k, Resistor_SMD:R_0201_0603Metric, F.Cu at (66.4, 77.3)
- added R124: 4.7k, Resistor_SMD:R_0201_0603Metric, F.Cu at (83.1, 76.9)
- added R125: 4.7k, Resistor_SMD:R_0201_0603Metric, F.Cu at (66.4, 76.6)
- added R126: 4.7k, Resistor_SMD:R_0201_0603Metric, F.Cu at (83.1, 79.2)
- added R127: 4.7k, Resistor_SMD:R_0201_0603Metric, F.Cu at (66.4, 78.8)
- added R128: 4.7k, Resistor_SMD:R_0201_0603Metric, F.Cu at (73.6, 74.7)
- added R129: 4.7k, Resistor_SMD:R_0201_0603Metric, F.Cu at (56.9, 74.3)
- added R130: 4.7k, Resistor_SMD:R_0201_0603Metric, F.Cu at (73.6, 75.7)
- added R131: 4.7k, Resistor_SMD:R_0201_0603Metric, F.Cu at (56.9, 75.4)
- added R132: 4.7k, Resistor_SMD:R_0201_0603Metric, F.Cu at (75.7, 80.5)
- added R133: 4.7k, Resistor_SMD:R_0201_0603Metric, F.Cu at (59.0, 80.1)
- added R134: 4.7k, Resistor_SMD:R_0201_0603Metric, F.Cu at (76.5, 80.5)
- added R135: 4.7k, Resistor_SMD:R_0201_0603Metric, F.Cu at (59.8, 80.1)
- added R136: 4.7k, Resistor_SMD:R_0201_0603Metric, B.Cu at (75.0, 80.5)
- added R137: 4.7k, Resistor_SMD:R_0201_0603Metric, B.Cu at (58.3, 80.1)
- added R138: 4.7k, Resistor_SMD:R_0201_0603Metric, B.Cu at (75.7, 80.5)
- added R139: 4.7k, Resistor_SMD:R_0201_0603Metric, B.Cu at (59.0, 80.1)
- added R140: 4.7k, Resistor_SMD:R_0201_0603Metric, B.Cu at (76.5, 80.5)
- added R141: 4.7k, Resistor_SMD:R_0201_0603Metric, B.Cu at (59.8, 80.1)
- added R142: 4.7k, Resistor_SMD:R_0201_0603Metric, F.Cu at (75.0, 80.5)
- added R143: 4.7k, Resistor_SMD:R_0201_0603Metric, F.Cu at (58.3, 80.1)
- added R144: 470, Resistor_SMD:R_0201_0603Metric, F.Cu at (85.9, 79.0)
- added R145: 470, Resistor_SMD:R_0201_0603Metric, F.Cu at (69.2, 78.7)
- added R146: 470, Resistor_SMD:R_0201_0603Metric, F.Cu at (85.9, 77.3)
- added R147: 470, Resistor_SMD:R_0201_0603Metric, F.Cu at (69.2, 76.9)
- added R148: 1k, Resistor_SMD:R_0201_0603Metric, B.Cu at (100.2, 96.8)
- added R149: 1k, Resistor_SMD:R_0201_0603Metric, B.Cu at (99.4, 96.8)
- added R150: 1k, Resistor_SMD:R_0201_0603Metric, B.Cu at (98.6, 96.9)
- added R151: 200, Resistor_SMD:R_0201_0603Metric, B.Cu at (97.8, 96.9)
- added R152: 200, Resistor_SMD:R_0201_0603Metric, B.Cu at (97.0, 96.9)
- added R153: 200, Resistor_SMD:R_0201_0603Metric, B.Cu at (96.2, 96.9)
- added R154: 1k, Resistor_SMD:R_0201_0603Metric, B.Cu at (95.3, 96.9)
- added R155: 39k, Resistor_SMD:R_0201_0603Metric, F.Cu at (128.2, 73.2)
- added R156: 470, Resistor_SMD:R_0201_0603Metric, F.Cu at (148.8, 116.4)
- added R157: 1k, Resistor_SMD:R_0201_0603Metric, F.Cu at (148.8, 115.0)
- added R158: 100k, Resistor_SMD:R_0201_0603Metric, F.Cu at (148.8, 113.3)
- added R159: 100, Resistor_SMD:R_0201_0603Metric, F.Cu at (144.6, 112.4)
- added R160: 22k, Resistor_SMD:R_0201_0603Metric, F.Cu at (148.8, 111.9)
- added R161: 1k, Resistor_SMD:R_0201_0603Metric, F.Cu at (151.6, 109.2)
- added R162: 100k, Resistor_SMD:R_0201_0603Metric, F.Cu at (154.4, 109.2)
- added R163: 100k, Resistor_SMD:R_0201_0603Metric, F.Cu at (153.3, 109.2)
- added R164: 100k, Resistor_SMD:R_0201_0603Metric, F.Cu at (152.6, 109.2)
- added R165: 100k, Resistor_SMD:R_0201_0603Metric, F.Cu at (150.9, 109.2)
- added R166: 100k, Resistor_SMD:R_0201_0603Metric, F.Cu at (150.1, 109.2)
- added R167: 0Ω, Resistor_SMD:R_0201_0603Metric, F.Cu at (129.7, 108.5)
- added R168: 10k, Resistor_SMD:R_0201_0603Metric, F.Cu at (131.0, 109.4)
- added R169: 100k, Resistor_SMD:R_0201_0603Metric, F.Cu at (56.4, 104.5)
- added R170: 100k, Resistor_SMD:R_0201_0603Metric, F.Cu at (56.4, 106.0)
- added R171: 100k, Resistor_SMD:R_0201_0603Metric, F.Cu at (56.4, 107.7)
- added R172: 100k, Resistor_SMD:R_0201_0603Metric, F.Cu at (56.4, 109.5)
- added R173: 0Ω, Resistor_SMD:R_0201_0603Metric, F.Cu at (117.0, 125.2)
- added R174: 0Ω, Resistor_SMD:R_0201_0603Metric, F.Cu at (121.0, 124.8)
- added R175: 0Ω, Resistor_SMD:R_0201_0603Metric, F.Cu at (117.1, 103.6)
- added R176: 10k, Resistor_SMD:R_0201_0603Metric, F.Cu at (116.4, 103.6)
- added R177: 120Ω, Resistor_SMD:R_0201_0603Metric, B.Cu at (100.8, 105.1)
- added R178: 240Ω, Resistor_SMD:R_0201_0603Metric, F.Cu at (116.1, 117.6)
- added R179: 240Ω, Resistor_SMD:R_0201_0603Metric, F.Cu at (116.0, 120.0)
- added R180: 51k, Resistor_SMD:R_0201_0603Metric, F.Cu at (141.8, 127.7)
- added R181: 6.3k, Resistor_SMD:R_0201_0603Metric, F.Cu at (143.4, 127.7)
- added R182: 200k, Resistor_SMD:R_0201_0603Metric, F.Cu at (141.9, 133.6)
- added R183: 14k, Resistor_SMD:R_0201_0603Metric, F.Cu at (142.0, 129.4)
- added R184: 100k, Resistor_SMD:R_0201_0603Metric, B.Cu at (142.5, 129.7)
- added R185: 100k, Resistor_SMD:R_0201_0603Metric, B.Cu at (143.5, 134.4)
- added R186: 14k, Resistor_SMD:R_0201_0603Metric, F.Cu at (141.8, 116.2)
- added R187: 75k, Resistor_SMD:R_0201_0603Metric, F.Cu at (141.7, 114.2)
- added R188: 24k, Resistor_SMD:R_0201_0603Metric, F.Cu at (143.2, 114.2)
- added R189: 200k, Resistor_SMD:R_0201_0603Metric, F.Cu at (141.6, 120.3)
- added R190: 200k, Resistor_SMD:R_0201_0603Metric, F.Cu at (132.4, 133.5)
- added R191: 14k, Resistor_SMD:R_0201_0603Metric, F.Cu at (132.7, 129.1)
- added R192: 27k, Resistor_SMD:R_0201_0603Metric, F.Cu at (132.5, 127.4)
- added R193: 5.1k, Resistor_SMD:R_0201_0603Metric, F.Cu at (134.0, 127.4)
- added R194: 0Ω, custom footprints:RF_Select_0201_L_Shape, F.Cu at (58.0, 116.8)
- added R195: 100k, Resistor_SMD:R_0201_0603Metric, F.Cu at (54.6, 92.5)
- added R196: 1k, Resistor_SMD:R_0201_0603Metric, F.Cu at (59.1, 92.5)
- added R197: 100k, Resistor_SMD:R_0201_0603Metric, F.Cu at (100.7, 87.6)
- added R198: 100k, Resistor_SMD:R_0201_0603Metric, F.Cu at (100.7, 89.1)
- added R199: 10k, Resistor_SMD:R_0201_0603Metric, F.Cu at (94.9, 87.6)
- added R200: 10k, Resistor_SMD:R_0402_1005Metric, F.Cu at (103.0, 80.3)
- added R201: 10k, Resistor_SMD:R_0402_1005Metric, F.Cu at (104.1, 80.3)
- added R202: 0Ω, Resistor_SMD:R_0402_1005Metric, F.Cu at (114.6, 79.5)
- added R203: 0Ω, Resistor_SMD:R_0402_1005Metric, B.Cu at (104.5, 72.6)
- added RJ1: HR911130A, easyeda:RJ45-TH_HR911130A, F.Cu at (78.4, 60.9)
- added RJ2: HR911130A, easyeda:RJ45-TH_HR911130A, F.Cu at (60.1, 60.9)
- added TP1: TestPoint, TestPoint:TestPoint_Pad_D1.0mm, F.Cu at (153.7, 107.0)
- added TP2: TestPoint, TestPoint:TestPoint_Pad_D1.0mm, F.Cu at (151.7, 106.9)
- added TP3: DCDC1, TestPoint:TestPoint_Pad_D1.0mm, F.Cu at (120.6, 109.4)
- added TP4: DCDC1, TestPoint:TestPoint_Pad_D1.0mm, F.Cu at (120.6, 111.5)
- added TP5: BT-UART0_RX, TestPoint:TestPoint_Pad_D1.0mm, F.Cu at (78.1, 116.8)
- added TP6: BT-UART0_TX, TestPoint:TestPoint_Pad_D1.0mm, F.Cu at (76.2, 117.7)
- added U1: GT-USB-7010ASV, easyeda:USB-C-SMD_G-SWITCH_GT-USB-7010ASV, F.Cu at (150.8, 122.7)
- added U10: AXP717B, easyeda:QFN-52_L6.0-W6.0-P0.40-TL-EP4.5, F.Cu at (126.6, 112.3)
- added U11: AXP323, custom footprints:AXP323, F.Cu at (116.9, 106.6)
- added U12: K4UBE3D4AB-MGCL, easyeda:FBGA-200_L14.5-W10.0_RS1G32LF4D2BDS-53BT, F.Cu at (107.9, 118.8)
- added U13: AFC11-S22ICA-00, easyeda:FPC-SMD_22P-P1.00_AFC11-S22ICC-00, F.Cu at (66.3, 102.3)
- added U14: RTL8211F-CG, easyeda:WQFN-40_L5.0-W5.0-P0.4-BL-EP, F.Cu at (77.6, 76.2)
- added U15: RTL8211F-CG, easyeda:WQFN-40_L5.0-W5.0-P0.4-BL-EP, F.Cu at (61.0, 75.9)
- added U16: HD3SS3202IRSVR, easyeda:UQFN-16_L2.6-W1.8-P0.40-BL, F.Cu at (97.4, 87.4)
- added U17: X3113WVS-36-9TV01, easyeda:CONN-SMD_X3113WVS-36-9TV01, F.Cu at (103.5, 74.5)
- added U18: HC-USB3.0-L168-WP, easyeda:USB-TH_USB3.0-A, F.Cu at (132.3, 61.5)
- added U19: ~, custom footprints:M8800DS2-40, F.Cu at (67.9, 118.5)
- added U21: CH217K, easyeda:SOT-23-6_L2.9-W1.6-P0.95-LS2.8-BL, F.Cu at (128.2, 70.6)
- added U22: CH334F_C5187527, easyeda:QFN-24_L4.0-W4.0-P0.50-BL-EP2.8, F.Cu at (123.5, 73.7)
- added U24: AFC11-S22ICA-00, easyeda:FPC-SMD_22P-P1.00_AFC11-S22ICC-00, F.Cu at (61.3, 102.2)
- added U25: AFC11-S22ICA-00, easyeda:FPC-SMD_22P-P1.00_AFC11-S22ICC-00, F.Cu at (71.6, 102.2)
- added U26: AFC11-S22ICA-00, easyeda:FPC-SMD_22P-P1.00_AFC11-S22ICC-00, F.Cu at (77.1, 102.2)
- added U3: AP64500SP-13, easyeda:SO-8_L4.9-W3.9-P1.27-LS6.0-BL-EP, F.Cu at (129.7, 130.5)
- added U4: STUSB4500QTR, easyeda:QFN-24_L4.0-W4.0-P0.50-BL-EP2.8, F.Cu at (152.1, 112.6)
- added U5: AP64350SP-13, easyeda:SO-8_L4.9-W3.9-P1.27-LS6.0-BL-EP, F.Cu at (139.0, 130.6)
- added U6: AP64500SP-13, easyeda:SO-8_L4.9-W3.9-P1.27-LS6.0-BL-EP, F.Cu at (138.8, 117.4)
- added U8: T527M00X0DCH, easyeda:BGA-664_L17.0-W17.0_T527, F.Cu at (94.8, 102.3)
- added U9: SY8089A1AAC, easyeda:TSOT-23-5_L2.9-W1.6-P0.95-LS2.8-BR, F.Cu at (120.4, 127.0)
- added USB1: Double layer DIP 90° black, easyeda:USB-A-TH_USB-M-51, F.Cu at (114.3, 61.8)
- added USB2: Double layer DIP 90° black, easyeda:USB-A-TH_USB-M-51, F.Cu at (96.3, 61.8)
- added X1: 25MHz, Crystal:Crystal_SMD_2520-4Pin_2.5x2.0mm, F.Cu at (84.2, 74.7)
- added X2: 25MHz, Crystal:Crystal_SMD_2520-4Pin_2.5x2.0mm, F.Cu at (67.5, 74.4)
- added X3: SMD-3225_4P12M12PF10PPM, easyeda:CRYSTAL-SMD_4P-L3.2-W2.5-BL, F.Cu at (123.8, 68.3)
Routing:
- net /T527/MCSIA-D1N: track 0.00 -> 37.6 mm
- net /T527/MCSIA-D0P: track 0.00 -> 37.5 mm
- net /T527/MCSIA-D0N: track 0.00 -> 36.0 mm
- net /T527/MCSIA-D1P: track 0.00 -> 35.5 mm
- net /T527/MCSIC-D0P: track 0.00 -> 27.3 mm
- net /T527/MCSIC-D0N: track 0.00 -> 25.9 mm
- net /T527/HCEC: track 0.00 -> 4.65 mm
- net /T527/HTXCP: track 0.00 -> 4.62 mm
- net /T527/HSCL: track 0.00 -> 4.44 mm
- net /T527/HTXCN: track 0.00 -> 4.41 mm
- net /T527/HTX0N: track 0.00 -> 4.41 mm
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Other:
- board outline added: 105 x 85 mm
- copper layers 2 -> 6

Commit message: started routing
Parts:
- removed R138, R139, R140, R141, R142, R143: 4.7k, Resistor_SMD:R_0201_0603Metric
- removed U18: HC-USB3.0-L168-WP, easyeda:USB-TH_USB3.0-A
- added C144: 100nF, PCM_JLCPCB:C_0402, F.Cu at (157.0, 98.5)
- added C145: 100nF, PCM_JLCPCB:C_0402, F.Cu at (155.5, 96.3)
- added C146: 1nF, PCM_JLCPCB:C_0402, F.Cu at (163.2, 99.2)
- added C147: 33pF, PCM_JLCPCB:C_0402, F.Cu at (158.5, 97.2)
- added C148: 2.2uF, PCM_JLCPCB:C_0402, F.Cu at (162.2, 97.2)
- added C149: 100nF, PCM_JLCPCB:C_0402, F.Cu at (159.4, 96.0)
- added C150: 100nF, PCM_JLCPCB:C_0402, F.Cu at (160.1, 112.6)
- added C173: 100nF, Capacitor_SMD:C_0201_0603Metric, F.Cu at (96.0, 27.8)
- added CN1: PJ-327A0-SMT, easyeda:AUDIO-SMD_PJ-327A0-SMT, F.Cu at (158.7, 106.3)
- added H1: MountingHole, custom footprints:NP-mounting-hole, F.Cu at (53.5, 48.5)
- added R204: 10k, Resistor_SMD:R_0201_0603Metric, F.Cu at (97.6, 29.6)
- added R205: 10k, Resistor_SMD:R_0201_0603Metric, F.Cu at (89.3, 31.9)
- added R47: 1kΩ, PCM_JLCPCB:R_0402, F.Cu at (157.9, 98.5)
- added R48: 1kΩ, PCM_JLCPCB:R_0402, F.Cu at (157.3, 96.3)
- added R49: 2kΩ, PCM_JLCPCB:R_0402, F.Cu at (160.3, 97.2)
- added R50: 47kΩ, PCM_JLCPCB:R_0402, F.Cu at (155.8, 112.2)
- added R51: 22Ω, PCM_JLCPCB:R_0402, F.Cu at (161.2, 96.0)
- added R52: 22Ω, PCM_JLCPCB:R_0402, F.Cu at (158.2, 112.6)
- added R53: 1MΩ, PCM_JLCPCB:R_0402, F.Cu at (153.9, 112.2)
- added R54: 100kΩ, PCM_JLCPCB:R_0402, F.Cu at (159.6, 98.5)
- added R55: 0Ω, PCM_JLCPCB:R_0402, F.Cu at (158.8, 98.5)
- added U2: GD25LQ128EWIGR, easyeda:WSON-8_L6.0-W5.0-P1.27-BL-EP, F.Cu at (93.4, 30.9)
- added USB4: HC-USB3.0-L168-WJ, easyeda:USB-3.0-A-TH_HC-USB3.0-L168-WJ, F.Cu at (140.3, 56.8)
- C1, C14, C15, C251, C252, C267, Q3, R136, R137, R184, R185: moved to F.Cu
- C186, C256, C257, R199: moved to B.Cu
- J2: footprint Connector_PinHeader_1.27mm:PinHeader_1x02_P1.27mm_Vertical -> Connector_PinHeader_2.54mm:PinHeader_1x02_P2.54mm_Vertical
- moved J2 60.9 mm to (150.7, 50.6)
- moved C257 22.2 mm to (106.7, 66.4), turned to -90 degrees
- moved D3 22.2 mm to (149.7, 129.7), turned to 0 degrees
- moved C159 21.3 mm to (136.0, 88.3)
- moved C184 21.3 mm to (79.5, 106.8), turned to -90 degrees
- moved C256 21.1 mm to (107.6, 66.3), turned to -90 degrees
- moved C186 20.0 mm to (108.5, 66.3), turned to -90 degrees
- moved R172 19.5 mm to (75.5, 105.3), turned to 90 degrees
- moved C9 17.9 mm to (148.1, 128.2), turned to 0 degrees
- moved U22 17.4 mm to (108.3, 65.1), turned to 90 degrees
- moved C165 16.9 mm to (136.0, 95.0)
- moved R159 16.6 mm to (149.9, 128.2), turned to 180 degrees
- moved C183 15.8 mm to (74.1, 106.8), turned to -90 degrees
- moved Q2 15.4 mm to (148.2, 126.0), turned to 90 degrees
- moved R109 15.4 mm to (148.7, 89.8)
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Connections:
- net /T527/DSI0-SCL renamed /T527/Disp0-SCL
- net /T527/DSI0-SDA renamed /T527/Disp0-SDA
- net /T527/DSI1-SCL renamed /T527/Disp1-SCL
- net /T527/DSI1-SDA renamed /T527/Disp1-SDA
- net /ethernet 1/GM_MDIN0 renamed /ethernet 1/GM_MDI0N
- net /ethernet 1/GM_MDIN1 renamed /ethernet 1/GM_MDI1N
- net /ethernet 1/GM_MDIN2 renamed /ethernet 1/GM_MDI2N
- net /ethernet 1/GM_MDIN3 renamed /ethernet 1/GM_MDI3N
- net /ethernet 1/GM_MDIP0 renamed /ethernet 1/GM_MDI0P
- net /ethernet 1/GM_MDIP1 renamed /ethernet 1/GM_MDI1P
- net /ethernet 1/GM_MDIP2 renamed /ethernet 1/GM_MDI2P
- net /ethernet 1/GM_MDIP3 renamed /ethernet 1/GM_MDI3P
- net /ethernet0/GM_MDIN0 renamed /ethernet0/GM_MDI0N
- net /ethernet0/GM_MDIN1 renamed /ethernet0/GM_MDI1N
- net /ethernet0/GM_MDIN2 renamed /ethernet0/GM_MDI2N
- net /ethernet0/GM_MDIN3 renamed /ethernet0/GM_MDI3N
- net /ethernet0/GM_MDIP0 renamed /ethernet0/GM_MDI0P
- net /ethernet0/GM_MDIP1 renamed /ethernet0/GM_MDI1P
- net /ethernet0/GM_MDIP2 renamed /ethernet0/GM_MDI2P
- net /ethernet0/GM_MDIP3 renamed /ethernet0/GM_MDI3P
- net Net-(D10-IN1) renamed /usb/USB2.0-4_DN
- net Net-(D10-IN2) renamed /usb/USB2.0-4_DP
- net Net-(D10-IN3) renamed /usb/USB2.0-3_DP
- net Net-(D10-IN4) renamed /usb/USB2.0-3_DN
- net Net-(D11-IN1) renamed /usb/USB2.0-2_DN
- net Net-(D11-IN2) renamed /usb/USB2.0-2_DP
- net Net-(D11-IN3) renamed /usb/USB2.0-1_DN
- net Net-(D11-IN4) renamed /usb/USB2.0-1_DP
- U16 pad 1: /T527/PCIE-TX0-DN -> /T527/PCIE-TX0-DP
- U16 pad 10: /pcie&usb3/USB3-TX0-DP -> /pcie&usb3/USB3-TX0-DN
- U16 pad 11: /pcie&usb3/PCIE_B-RX0-DN -> /pcie&usb3/PCIE_B-RX0-DP
- U16 pad 12: /pcie&usb3/PCIE_B-RX0-DP -> /pcie&usb3/PCIE_B-RX0-DN
- U16 pad 13: /pcie&usb3/PCIE_B-TX0-DN -> /pcie&usb3/PCIE_B-TX0-DP
- U16 pad 14: /pcie&usb3/PCIE_B-TX0-DP -> /pcie&usb3/PCIE_B-TX0-DN
- U16 pad 16: /T527/PCIE-TX0-DP -> /T527/PCIE-TX0-DN
- U16 pad 4: /T527/PCIE-RX0-DP -> /T527/PCIE-RX0-DN
- U16 pad 5: /T527/PCIE-RX0-DN -> /T527/PCIE-RX0-DP
- U16 pad 7: /pcie&usb3/USB3-RX0-DN -> /pcie&usb3/USB3-RX0-DP
- U16 pad 8: /pcie&usb3/USB3-RX0-DP -> /pcie&usb3/USB3-RX0-DN
- U16 pad 9: /pcie&usb3/USB3-TX0-DN -> /pcie&usb3/USB3-TX0-DP
- U8 pad E24: /T527/USB1-DM -> /T527/USB1-DN
- U8 pad U28: unconnected-(U8D-PC4-PadU28) -> /T527/SPI0_DI
- U8 pad U29: unconnected-(U8D-PC3-PadU29) -> /T527/SPI0_CS
- U8 pad U30: unconnected-(U8D-PC2-PadU30) -> /T527/SPI0_DO
- U8 pad V31: unconnected-(U8D-PC11-PadV31) -> /T527/SPI0_CLK
Routing:
- net /T527/HTX2N: track 0.00 -> 74.4 mm
- net /T527/HTX2P: track 0.00 -> 74.2 mm
- net /T527/HTX1N: track 0.00 -> 72.3 mm
- net /T527/HTX1P: track 0.00 -> 72.1 mm
- net /T527/HTX0P: track 0.00 -> 71.2 mm
- net /T527/HSDA: track 0.00 -> 67.6 mm, vias 0 -> 2
- net /T527/HTX0N: track 4.41 -> 71.4 mm
- net /T527/USB2-DN: track 0.00 -> 66.2 mm, vias 0 -> 1
- net /T527/HHPD: track 0.00 -> 66.1 mm, vias 0 -> 2
- net /T527/HTXCP: track 4.62 -> 70.5 mm
- net /T527/HTXCN: track 4.41 -> 69.6 mm
- net /T527/USB2-DP: track 0.00 -> 64.8 mm, vias 0 -> 1
- net /T527/HCEC: track 4.65 -> 69.2 mm, vias 0 -> 2
- net /T527/HSCL: track 4.44 -> 67.8 mm, vias 0 -> 2
- net /pcie&usb3/USB3-RX0-DP: track 0.00 -> 58.9 mm
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- added copper zone on F.Cu, net /power input/VBUS_MAIN
- added copper zone on F.Cu, net /power input/V_MAIN
- added copper zone on F.Cu, net GND
Other:
- board size 105 x 85 mm -> 115 x 90 mm
- board text added: "DP"
- board text added: "DSI0"
- board text added: "DSI1"
- board text added: "HDMI"
- board text added: "MCSIA"
- board text added: "MCSIB"
- board text added: "MCSIC"
- board text added: "MCSID"

Commit message: finsihed more routing
Parts:
- added C304: 12pF, Capacitor_SMD:C_0201_0603Metric, F.Cu at (94.8, 112.3)
- added C305: 12pF, Capacitor_SMD:C_0201_0603Metric, F.Cu at (93.1, 112.3)
- added C306: 12pF, Capacitor_SMD:C_0201_0603Metric, F.Cu at (90.2, 115.2)
- added C307: 12pF, Capacitor_SMD:C_0201_0603Metric, F.Cu at (88.7, 115.2)
- added M1: Fan&Heatsink_40x40mm, custom footprints:custom_heatsink&fan_40x40mm, B.Cu at (136.7, 114.0)
- added R206: 10M, Resistor_SMD:R_0201_0603Metric, F.Cu at (89.4, 112.5)
- added R207: 4.3k, Resistor_SMD:R_0201_0603Metric, B.Cu at (81.5, 103.9)
- added R208: 6.8k, Resistor_SMD:R_0201_0603Metric, B.Cu at (83.0, 103.9)
- added R209: 10k, Resistor_SMD:R_0201_0603Metric, B.Cu at (83.0, 105.0)
- added R210: 10k, Resistor_SMD:R_0201_0603Metric, B.Cu at (81.5, 105.0)
- added R211: 10k, Resistor_SMD:R_0201_0603Metric, B.Cu at (83.0, 106.1)
- added R212: 10k, Resistor_SMD:R_0201_0603Metric, B.Cu at (81.5, 106.1)
- added R213: 10k, Resistor_SMD:R_0201_0603Metric, B.Cu at (82.5, 107.6)
- added R214: 10k, Resistor_SMD:R_0201_0603Metric, B.Cu at (82.5, 108.4)
- added X4: 25MHz, Crystal:Crystal_SMD_3225-4Pin_3.2x2.5mm, F.Cu at (93.9, 114.5)
- added X5: SC-20S32.768kHz20PPM9pF, easyeda:OSC-SMD_L2.0-W1.2, F.Cu at (89.4, 113.8)
- C261, C262, C263, C264: moved to F.Cu
- C300, Q4, R195, R196: moved to B.Cu
- R197: value 100k -> 1k
- moved C173 80.7 mm to (119.3, 105.0), turned to 90 degrees
- moved R204 78.3 mm to (118.6, 105.1)
- moved R205 78.3 mm to (110.2, 107.4)
- moved U2 78.3 mm to (114.4, 106.3)
- moved R202 23.6 mm to (92.7, 68.6), turned to 0 degrees
- moved C257 17.1 mm to (121.5, 75.0), turned to -45 degrees
- moved C179 17.0 mm to (96.2, 77.4), turned to 180 degrees
- moved C256 16.5 mm to (122.1, 74.3), turned to -45 degrees
- moved C180 16.5 mm to (96.2, 69.5), turned to 180 degrees
- moved C178 16.2 mm to (96.1, 76.2), turned to 180 degrees
- moved C186 16.0 mm to (122.7, 73.6), turned to -45 degrees
- moved C172 15.6 mm to (96.2, 70.6), turned to 180 degrees
- moved U22 15.2 mm to (121.5, 72.7), turned to 135 degrees
- moved R155 15.1 mm to (131.6, 63.4), turned to -90 degrees
- moved C259 14.1 mm to (127.3, 70.8), turned to 45 degrees
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Connections:
- D13 pad 1: /power input/UART0_TX -> /T527/DBG_UART0_TX
- D13 pad 10: /power input/UART0_TX -> /T527/DBG_UART0_TX
- D13 pad 2: /power input/DP -> /T527/DBG_DP
- D13 pad 4: /power input/DN -> /T527/DBG_DN
- D13 pad 5: /power input/UART0_RX -> /T527/DBG_UART0_RX
- D13 pad 6: /power input/UART0_RX -> /T527/DBG_UART0_RX
- D13 pad 7: /power input/DN -> /T527/DBG_DN
- D13 pad 9: /power input/DP -> /T527/DBG_DP
- TP3 pad 1: /power/PMU-SDA -> /T527/PMU-SDA
- TP4 pad 1: /power/PMU-SCK -> /T527/PMU-SCK
- U1 pad A6: /power input/DP -> /T527/DBG_DP
- U1 pad A7: /power input/DN -> /T527/DBG_DN
- U1 pad A8: /power input/UART0_TX -> /T527/DBG_UART0_TX
- U1 pad B6: /power input/DP -> /T527/DBG_DP
- U1 pad B7: /power input/DN -> /T527/DBG_DN
- U1 pad B8: /power input/UART0_RX -> /T527/DBG_UART0_RX
- U10 pad 51: /power/PMU-SDA -> /T527/PMU-SDA
- U10 pad 52: /power/PMU-SCK -> /T527/PMU-SCK
- U11 pad 5: /power/PMU-SCK -> /T527/PMU-SCK
- U11 pad 6: /power/PMU-SDA -> /T527/PMU-SDA
- U17 pad 29: /pcie&usb3/PCIE0-WAKEN  -> /T527/PCIE0-WAKEN
- U8 pad A16: /T527/PCIE0-PERSTN  -> /T527/PCIE0-PERSTN
- U8 pad A2: unconnected-(U8C-PE7-PadA2) -> /T527/LED-EN-B
- U8 pad A24: /T527/DP -> /T527/DBG_DP
- U8 pad A3: unconnected-(U8C-PE6-PadA3) -> /T527/LED-EN-C
- U8 pad AM11: unconnected-(U8A-X32KOUT-PadAM11) -> /T527/X32KOUT
- U8 pad AM12: unconnected-(U8A-X32KIN-PadAM12) -> /T527/X32KIN
- U8 pad AM13: unconnected-(U8A-DXIN-PadAM13) -> /T527/DXIN
- U8 pad AN13: unconnected-(U8A-DXOUT-PadAN13) -> /T527/DXOUT
- U8 pad AN5: unconnected-(U8C-PL1-PadAN5) -> /T527/PMU-SDA
- U8 pad AN6: unconnected-(U8C-PL0-PadAN6) -> /T527/PMU-SCK
- U8 pad B1: unconnected-(U8C-PE9-PadB1) -> /T527/LED-EN-D
- U8 pad B15: unconnected-(U8D-PH13-PadB15) -> /ETH0.RGMII-INTB
- U8 pad B2: unconnected-(U8C-PE8-PadB2) -> /T527/POWER-EN-D
- U8 pad B24: /T527/DN -> /T527/DBG_DN
- U8 pad B3: unconnected-(U8C-PE5-PadB3) -> /T527/POWER-EN-C
- U8 pad C1: unconnected-(U8C-PE12-PadC1) -> /T527/SCL-A
- U8 pad C2: unconnected-(U8C-PE10-PadC2) -> /T527/POWER-EN-A
- U8 pad C3: unconnected-(U8C-PE4-PadC3) -> /T527/SDA-C
- U8 pad C4: unconnected-(U8C-PE1-PadC4) -> /T527/SCL-B
- U8 pad D16: unconnected-(U8D-PH8-PadD16) -> /ETH0.RGMII-PHYRSTB
- U8 pad E4: unconnected-(U8C-PE3-PadE4) -> /T527/SCL-C
- U8 pad E5: unconnected-(U8C-PE2-PadE5) -> /T527/SDA-B
- U8 pad E6: unconnected-(U8C-PE0-PadE6) -> /T527/POWER-EN-B
- U8 pad G4: unconnected-(U8D-PJ10-PadG4) -> /ETH1.RGMII-PHYRSTB
- U8 pad G6: unconnected-(U8C-PE13-PadG6) -> /T527/SDA-A
- U8 pad J1: unconnected-(U8D-PJ16-PadJ1) -> /ETH1.RGMII-INTB
- U8 pad J7: unconnected-(U8C-PE11-PadJ7) -> /T527/LED-EN-A
- U8 pad L31: unconnected-(U8D-PD22-PadL31) -> /T527/Disp0-SCL
- U8 pad L32: unconnected-(U8D-PD23-PadL32) -> /T527/Disp0-SDA
- U8 pad L7: unconnected-(U8C-PE14-PadL7) -> /T527/SCL-D
- U8 pad N7: unconnected-(U8C-PE15-PadN7) -> /T527/SDA-D
- U8 pad R28: unconnected-(U8C-PB9-PadR28) -> /T527/DBG_UART0_TX
- U8 pad R29: unconnected-(U8C-PB10-PadR29) -> /T527/DBG_UART0_RX
- U8 pad R30: unconnected-(U8C-PB11-PadR30) -> /T527/Disp1-SCL
- U8 pad R31: unconnected-(U8C-PB12-PadR31) -> /T527/Disp1-SDA
- U8 pad V2: unconnected-(U8A-LRADC1-PadV2) -> Net-(U8A-LRADC1)
- U8 pad V3: unconnected-(U8A-LRADC0-PadV3) -> Net-(U8A-LRADC0)
- U8 pad W1: unconnected-(U8D-GPADC0-PadW1) -> /T527/BOOT_SEL_ADC
- U8 pad W2: unconnected-(U8D-GPADC1-PadW2) -> /T527/DDR-PARA-SEL-ADC1
- U8 pad W3: unconnected-(U8D-GPADC2-PadW3) -> /T527/DDR-PARA-SEL-ADC2
Routing:
- net /T527/DBG_DP: track 0.00 -> 88.7 mm, vias 0 -> 2
- net /T527/DBG_DN: track 0.00 -> 87.9 mm, vias 0 -> 2
- net Net-(J2-Pin_2): track 0.00 -> 73.0 mm, vias 0 -> 1
- net /T527/SDC0-DET: track 0.00 -> 51.6 mm, vias 0 -> 2
- net /ETH1.RGMII-PHYRSTB: track 2.13 -> 47.7 mm, vias 0 -> 2
- net /T527/Disp1-SDA: track 0.00 -> 44.0 mm, vias 0 -> 2
- net /T527/Disp1-SCL: track 0.00 -> 43.0 mm, vias 0 -> 2
- net /T527/AP-WAKE-BT: track 0.00 -> 42.8 mm, vias 0 -> 2
- net /T527/SDA-A: track 0.00 -> 41.0 mm, vias 0 -> 2
- net /T527/LED-EN-A: track 0.00 -> 40.1 mm, vias 0 -> 2
- net /T527/BT-WAKE-AP: track 0.00 -> 40.0 mm, vias 0 -> 2
- net /ETH1.RGMII-INTB: track 3.14 -> 43.1 mm, vias 0 -> 2
- net /T527/POWER-EN-A: track 0.00 -> 39.8 mm, vias 0 -> 2
- net /T527/Disp0-SDA: track 0.00 -> 38.8 mm, vias 0 -> 2
- net /T527/Disp0-SCL: track 0.00 -> 38.5 mm, vias 0 -> 2
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- added copper zone on B.Cu, net GND
- added copper zone on In1.Cu, net GND
- added copper zone on In4.Cu, net GND
Other:
- board text added: "0:PCIe 1:USB3"
