File: PCB/Artificer A1 Board Rev 0.1/Artificer A1 Board Rev 0.1.kicad_pcb (KiCad board)
At the start: 6 copper layers, 115 x 90 mm, 385 parts, among them CN1 PJ-327A0-SMT, J1 Conn_02x20_Odd_Even, J2 Conn_01x02, M1 Fan&Heatsink_40x40mm, Q1 AON3419-TP, Q2 AON3419-TP, Q3 AO3401A, Q4 2SK3018, Q6 AO3401A, Q7 AO3401A, U1 GT-USB-7010ASV, U10 AXP717B, U11 AXP323, U12 K4UBE3D4AB-MGCL, U13 AFC11-S22ICA-00, U14 RTL8211F-CG, U15 RTL8211F-CG, U16 HD3SS3202IRSVR, U17 X3113WVS-36-9TV01, U2 GD25LQ128EWIGR, U21 CH217K, U22 CH334F_C5187527, U24 AFC11-S22ICA-00, U25 AFC11-S22ICA-00, U26 AFC11-S22ICA-00, U3 AP64500SP-13, U4 STUSB4500QTR, U5 AP64350SP-13, U6 AP64500SP-13, U8 T527M00X0DCH, U9 SY8089A1AAC, X1 25MHz, X2 25MHz, X3 SMD-3225_4P12M12PF10PPM, X4 25MHz, X5 SC-20S32.768kHz20PPM9pF

Commit message: more routing and decoupling
Parts:
- removed C198, C199, C200, C201, C202, C203, C206: 100nF, Capacitor_SMD:C_0201_0603Metric
- added C308: 2.2uF, Capacitor_SMD:C_0201_0603Metric, B.Cu at (109.4, 123.8)
- added C309: 100nF, Capacitor_SMD:C_0201_0603Metric, B.Cu at (101.6, 115.0)
- added C310: 2.2uF, Capacitor_SMD:C_0201_0603Metric, B.Cu at (108.2, 115.0)
- added C311: 2.2uF, Capacitor_SMD:C_0201_0603Metric, B.Cu at (103.0, 115.0)
- added C312: 2.2uF, Capacitor_SMD:C_0201_0603Metric, B.Cu at (107.5, 123.8)
- added C313: 2.2uF, Capacitor_SMD:C_0201_0603Metric, B.Cu at (103.0, 123.8)
- added C314: 2.2uF, Capacitor_SMD:C_0201_0603Metric, B.Cu at (102.2, 116.5)
- added C315: 2.2uF, Capacitor_SMD:C_0201_0603Metric, B.Cu at (108.7, 116.7)
- added C316: 2.2uF, Capacitor_SMD:C_0201_0603Metric, B.Cu at (102.3, 122.2)
- added C317: 2.2uF, Capacitor_SMD:C_0201_0603Metric, B.Cu at (108.8, 122.2)
- added C318: 2.2uF, Capacitor_SMD:C_0201_0603Metric, B.Cu at (100.3, 119.4)
- added C319: 2.2uF, Capacitor_SMD:C_0201_0603Metric, B.Cu at (110.3, 118.9)
- added C320: 100nF, Capacitor_SMD:C_0201_0603Metric, B.Cu at (110.5, 123.5)
- added C321: 100nF, Capacitor_SMD:C_0201_0603Metric, B.Cu at (99.0, 118.2)
- added C322: 100nF, Capacitor_SMD:C_0201_0603Metric, B.Cu at (110.1, 115.0)
- added C323: 100nF, Capacitor_SMD:C_0201_0603Metric, B.Cu at (100.1, 115.0)
- added C324: 10uF, Capacitor_SMD:C_0402_1005Metric, B.Cu at (102.0, 119.8)
- added C325: 10uF, Capacitor_SMD:C_0402_1005Metric, B.Cu at (110.3, 119.8)
- added C326: 10uF, Capacitor_SMD:C_0402_1005Metric, B.Cu at (100.8, 103.8)
- added C327: 10uF, Capacitor_SMD:C_0402_1005Metric, B.Cu at (96.4, 107.0)
- added C328: 2.2uF, Capacitor_SMD:C_0201_0603Metric, B.Cu at (99.1, 103.2)
- added C329: 2.2uF, Capacitor_SMD:C_0201_0603Metric, B.Cu at (96.2, 106.2)
- added C330: 2.2uF, Capacitor_SMD:C_0201_0603Metric, B.Cu at (99.1, 103.9)
- added C331: 2.2uF, Capacitor_SMD:C_0201_0603Metric, B.Cu at (96.2, 105.4)
- added C332: 2.2uF, Capacitor_SMD:C_0201_0603Metric, B.Cu at (89.6, 106.9)
- added C333: 2.2uF, Capacitor_SMD:C_0201_0603Metric, B.Cu at (89.0, 109.0)
- added C334: 2.2uF, Capacitor_SMD:C_0201_0603Metric, B.Cu at (90.4, 103.9)
- added C335: 2.2uF, Capacitor_SMD:C_0201_0603Metric, B.Cu at (88.3, 108.9)
- added C336: 2.2uF, Capacitor_SMD:C_0201_0603Metric, B.Cu at (87.5, 108.9)
- added C337: 2.2uF, Capacitor_SMD:C_0201_0603Metric, B.Cu at (89.6, 103.9)
- added C338: 470nF, Capacitor_SMD:C_0201_0603Metric, B.Cu at (88.8, 106.9)
- added C339: 470nF, Capacitor_SMD:C_0201_0603Metric, B.Cu at (88.1, 106.9)
- added C340: 470nF, Capacitor_SMD:C_0201_0603Metric, B.Cu at (89.2, 105.8)
- added C341: 2.2uF, Capacitor_SMD:C_0201_0603Metric, B.Cu at (97.7, 99.3)
- added C342: 2.2uF, Capacitor_SMD:C_0201_0603Metric, B.Cu at (98.8, 106.5)
- added C343: 100nF, Capacitor_SMD:C_0201_0603Metric, B.Cu at (99.5, 106.5)
- added C344: 100nF, Capacitor_SMD:C_0201_0603Metric, B.Cu at (99.1, 104.7)
- added C345: 100nF, Capacitor_SMD:C_0201_0603Metric, B.Cu at (99.1, 105.4)
- added C346: 100nF, Capacitor_SMD:C_0201_0603Metric, B.Cu at (97.6, 105.4)
- added C347: 100nF, Capacitor_SMD:C_0201_0603Metric, B.Cu at (97.6, 106.2)
- added C348: 2.2uF, Capacitor_SMD:C_0201_0603Metric, B.Cu at (94.7, 101.0)
- added C349: 2.2uF, Capacitor_SMD:C_0201_0603Metric, B.Cu at (99.2, 98.6)
- added C350: 2.2uF, Capacitor_SMD:C_0201_0603Metric, B.Cu at (95.1, 99.8)
- added C351: 2.2uF, Capacitor_SMD:C_0201_0603Metric, B.Cu at (92.2, 98.7)
- added C352: 2.2uF, Capacitor_SMD:C_0201_0603Metric, B.Cu at (93.4, 97.6)
- added C356: 100nF, Capacitor_SMD:C_0201_0603Metric, B.Cu at (97.7, 100.1)
- added C357: 100nF, Capacitor_SMD:C_0201_0603Metric, B.Cu at (97.7, 98.6)
- added C358: 100nF, Capacitor_SMD:C_0201_0603Metric, B.Cu at (96.2, 99.3)
- added C359: 100nF, Capacitor_SMD:C_0201_0603Metric, B.Cu at (92.2, 99.4)
- added C360: 100nF, Capacitor_SMD:C_0201_0603Metric, B.Cu at (94.2, 97.6)
- added C363: 100nF, Capacitor_SMD:C_0201_0603Metric, B.Cu at (96.2, 98.6)
- added C364: 100nF, Capacitor_SMD:C_0201_0603Metric, B.Cu at (94.7, 98.7)
- added C365: 100nF, Capacitor_SMD:C_0201_0603Metric, B.Cu at (94.9, 97.6)
- added C374: 1uF, Capacitor_SMD:C_0201_0603Metric, B.Cu at (97.7, 101.6)
- added C375: 100nF, Capacitor_SMD:C_0201_0603Metric, B.Cu at (97.7, 102.3)
- added C376: 100nF, Capacitor_SMD:C_0201_0603Metric, B.Cu at (100.0, 110.3)
- added C377: 22uF, Capacitor_SMD:C_0603_1608Metric, B.Cu at (113.3, 107.3)
- added C378: 22uF, Capacitor_SMD:C_0603_1608Metric, B.Cu at (113.3, 109.8)
- added C379: 2.2uF, Capacitor_SMD:C_0201_0603Metric, B.Cu at (97.6, 103.1)
- added C380: 2.2uF, Capacitor_SMD:C_0201_0603Metric, B.Cu at (97.6, 103.8)
- added C381: 2.2uF, Capacitor_SMD:C_0201_0603Metric, B.Cu at (97.6, 104.6)
- added C382: 1uF, Capacitor_SMD:C_0201_0603Metric, B.Cu at (96.2, 103.1)
- added C383: 100nF, Capacitor_SMD:C_0201_0603Metric, B.Cu at (96.2, 103.8)
- added C384: 100nF, Capacitor_SMD:C_0201_0603Metric, B.Cu at (96.2, 104.6)
- added C385: 22uF, Capacitor_SMD:C_0603_1608Metric, B.Cu at (114.2, 104.7)
- added C386: 2.2uF, Capacitor_SMD:C_0201_0603Metric, B.Cu at (97.7, 100.8)
- added C387: 22uF, Capacitor_SMD:C_0603_1608Metric, B.Cu at (108.2, 103.2)
- added C388: 2.2uF, Capacitor_SMD:C_0201_0603Metric, B.Cu at (92.2, 100.2)
- added C389: 22uF, Capacitor_SMD:C_0603_1608Metric, B.Cu at (111.9, 102.9)
- added C390: 2.2uF, Capacitor_SMD:C_0201_0603Metric, B.Cu at (95.1, 102.2)
- added C391: 2.2uF, Capacitor_SMD:C_0201_0603Metric, B.Cu at (92.6, 101.7)
- added C392: 100nF, Capacitor_SMD:C_0201_0603Metric, B.Cu at (93.3, 101.7)
- added C393: 100nF, Capacitor_SMD:C_0201_0603Metric, B.Cu at (94.3, 102.2)
- added C394: 22uF, Capacitor_SMD:C_0603_1608Metric, B.Cu at (109.7, 105.5)
- added C395: 2.2uF, Capacitor_SMD:C_0201_0603Metric, B.Cu at (92.6, 103.2)
- added C396: 2.2uF, Capacitor_SMD:C_0201_0603Metric, B.Cu at (93.3, 103.2)
- added C397: 2.2uF, Capacitor_SMD:C_0201_0603Metric, B.Cu at (91.5, 102.0)
- added C398: 100nF, Capacitor_SMD:C_0201_0603Metric, B.Cu at (91.5, 102.8)
- added C399: 22uF, Capacitor_SMD:C_0603_1608Metric, B.Cu at (109.9, 108.3)
- added C400: 2.2uF, Capacitor_SMD:C_0201_0603Metric, B.Cu at (93.0, 104.3)
- added C401: 2.2uF, Capacitor_SMD:C_0201_0603Metric, B.Cu at (91.5, 103.6)
- added C402: 2.2uF, Capacitor_SMD:C_0201_0603Metric, B.Cu at (91.5, 104.3)
- added C403: 100nF, Capacitor_SMD:C_0201_0603Metric, B.Cu at (93.0, 105.1)
- added C404: 2.2uF, Capacitor_SMD:C_0201_0603Metric, B.Cu at (91.5, 105.1)
- added C405: 2.2uF, Capacitor_SMD:C_0201_0603Metric, B.Cu at (94.7, 105.8)
- added C406: 100nF, Capacitor_SMD:C_0201_0603Metric, B.Cu at (94.7, 105.0)
- added C407: 1uF, Capacitor_SMD:C_0201_0603Metric, B.Cu at (93.4, 99.8)
- added C408: 100nF, Capacitor_SMD:C_0201_0603Metric, B.Cu at (94.1, 99.8)
- added C409: 1uF, Capacitor_SMD:C_0201_0603Metric, B.Cu at (98.8, 99.7)
- added C410: 100nF, Capacitor_SMD:C_0201_0603Metric, B.Cu at (99.2, 102.4)
- added C411: 100nF, Capacitor_SMD:C_0201_0603Metric, B.Cu at (99.6, 99.7)
- added C412: 100nF, Capacitor_SMD:C_0201_0603Metric, B.Cu at (99.2, 100.8)
- added C413: 100nF, Capacitor_SMD:C_0201_0603Metric, B.Cu at (90.4, 99.8)
- added C414: 100nF, Capacitor_SMD:C_0201_0603Metric, B.Cu at (90.3, 98.7)
- added C415: 100nF, Capacitor_SMD:C_0201_0603Metric, B.Cu at (90.1, 102.0)
- added C416: 100nF, Capacitor_SMD:C_0201_0603Metric, B.Cu at (94.7, 106.5)
- added C417: 1uF, Capacitor_SMD:C_0201_0603Metric, B.Cu at (90.4, 100.6)
- added C418: 100nF, Capacitor_SMD:C_0201_0603Metric, B.Cu at (90.4, 101.3)
- added C419: 100nF, Capacitor_SMD:C_0201_0603Metric, B.Cu at (91.1, 98.7)
- added C420: 100nF, Capacitor_SMD:C_0201_0603Metric, B.Cu at (92.2, 97.9)
- added C421: 100nF, Capacitor_SMD:C_0201_0603Metric, B.Cu at (91.8, 107.0)
- added C422: 100nF, Capacitor_SMD:C_0201_0603Metric, B.Cu at (90.8, 107.0)
- added C423: 100nF, Capacitor_SMD:C_0201_0603Metric, B.Cu at (99.2, 101.7)
- added C424: 100nF, Capacitor_SMD:C_0201_0603Metric, B.Cu at (92.8, 106.6)
- added C425: 2.2uF, Capacitor_SMD:C_0201_0603Metric, B.Cu at (94.0, 107.3)
- added C426: 100nF, Capacitor_SMD:C_0201_0603Metric, B.Cu at (93.6, 106.2)
- added C427: 100nF, Capacitor_SMD:C_0201_0603Metric, B.Cu at (96.2, 100.1)
- added C428: 100nF, Capacitor_SMD:C_0201_0603Metric, B.Cu at (90.3, 105.4)
- added R215: 4.7k, Resistor_SMD:R_0201_0603Metric, F.Cu at (58.9, 107.1)
- added R216: 4.7k, Resistor_SMD:R_0201_0603Metric, F.Cu at (63.1, 106.8)
- added R217: 4.7k, Resistor_SMD:R_0201_0603Metric, F.Cu at (64.4, 107.2)
- added R218: 4.7k, Resistor_SMD:R_0201_0603Metric, F.Cu at (68.6, 106.8)
- added R219: 4.7k, Resistor_SMD:R_0201_0603Metric, F.Cu at (69.9, 107.2)
- added R220: 4.7k, Resistor_SMD:R_0201_0603Metric, F.Cu at (74.1, 106.8)
- added R221: 4.7k, Resistor_SMD:R_0201_0603Metric, F.Cu at (75.4, 107.2)
- added R222: 4.7k, Resistor_SMD:R_0201_0603Metric, F.Cu at (79.7, 106.8)
- added R223: 4.7k, Resistor_SMD:R_0201_0603Metric, F.Cu at (135.8, 88.4)
- added R224: 4.7k, Resistor_SMD:R_0201_0603Metric, F.Cu at (136.4, 92.5)
- added R225: 4.7k, Resistor_SMD:R_0201_0603Metric, F.Cu at (142.5, 95.5)
- added R226: 4.7k, Resistor_SMD:R_0201_0603Metric, F.Cu at (136.3, 99.0)
- added R227: 4.7k, Resistor_SMD:R_0201_0603Metric, F.Cu at (127.0, 108.0)
- added R228: 4.7k, Resistor_SMD:R_0201_0603Metric, F.Cu at (127.0, 106.0)
- added R229: 0Ω, Resistor_SMD:R_0201_0603Metric, B.Cu at (92.4, 108.8)
- added R230: 10k, Resistor_SMD:R_0201_0603Metric, F.Cu at (126.9, 105.0)
- added R231: 10k, Resistor_SMD:R_0201_0603Metric, F.Cu at (140.9, 102.9)
- added R232: 0Ω, Resistor_SMD:R_0201_0603Metric, B.Cu at (89.2, 105.0)
- added SW1: BOOT1, easyeda:SW-SMD_4P-L3.5-W3.0-P1.50-LS4.7, F.Cu at (54.0, 56.0)
- added SW2: RESET, easyeda:SW-SMD_4P-L3.5-W3.0-P1.50-LS4.7, F.Cu at (54.0, 64.0)
- C162, C163: value 100nF -> 10nF
- C173, C191, C192, R204, R205: moved to B.Cu
- C282: value 1uF -> 2.2uF
- C283: value 1uF -> 22uF; footprint Capacitor_SMD:C_0201_0603Metric -> Capacitor_SMD:C_0603_1608Metric
- C284: value 1uF -> 22uF; footprint Capacitor_SMD:C_0201_0603Metric -> Capacitor_SMD:C_0603_1608Metric; moved to B.Cu
- C285: value 1uF -> 2.2uF; moved to B.Cu
- C286: value 100nF -> 2.2uF
- R173: value 0Ω -> 1k
- R174: value 0Ω -> 100k
- R202: value 0Ω -> 10k; footprint Resistor_SMD:R_0402_1005Metric -> Resistor_SMD:R_0201_0603Metric
- moved J1 48.3 mm to (106.6, 130.2), turned to -90 degrees
- moved C285 23.2 mm to (96.2, 102.3), turned to 180 degrees
- moved C282 21.0 mm to (96.2, 100.9)
- moved C286 19.6 mm to (96.2, 101.6), turned to 180 degrees
- moved C284 16.0 mm to (106.8, 109.0), turned to 180 degrees
- moved C173 12.0 mm to (114.0, 94.2), turned to 0 degrees
- moved C283 10.2 mm to (106.8, 110.5)
- moved R204 10.1 mm to (115.0, 95.7)
- moved U2 9.78 mm to (111.8, 96.9)
- moved R205 9.67 mm to (107.7, 98.1)
- moved C288 9.49 mm to (102.0, 118.9)
- moved R213 6.89 mm to (87.8, 103.2), turned to -90 degrees
- moved R214 6.85 mm to (87.0, 103.2), turned to -90 degrees
- moved R210 3.03 mm to (84.5, 104.5)
- moved R207 3.00 mm to (84.5, 103.7)
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Connections:
- net /dram/SCKN-A renamed /dram/SCKA-N
- net /dram/SCKN-B renamed /dram/SCKB-N
- net /dram/SCKP-A renamed /dram/SCKA-P
- net /dram/SCKP-B renamed /dram/SCKB-P
- C282 pad 2: DCDC3 -> 323-DCDC1/2
- C283 pad 2: DCDC3 -> 323-DCDC1/2
- C284 pad 2: ALDO4 -> 323-DCDC1/2
- C285 pad 2: ALDO4 -> 323-DCDC1/2
- C286 pad 2: VDD06-DRAM -> 323-DCDC1/2
- J1 pad 1: unconnected-(J1-Pin_1-Pad1) -> VCC-3V3
- J1 pad 10: unconnected-(J1-Pin_10-Pad10) -> /T527/PL3
- J1 pad 11: unconnected-(J1-Pin_11-Pad11) -> /T527/PL4
- J1 pad 12: unconnected-(J1-Pin_12-Pad12) -> /T527/PL10
- J1 pad 13: unconnected-(J1-Pin_13-Pad13) -> /T527/PL5
- J1 pad 14: unconnected-(J1-Pin_14-Pad14) -> GND
- J1 pad 15: unconnected-(J1-Pin_15-Pad15) -> /T527/PL6
- J1 pad 16: unconnected-(J1-Pin_16-Pad16) -> /T527/PL7
- J1 pad 17: unconnected-(J1-Pin_17-Pad17) -> VCC-3V3
- J1 pad 18: unconnected-(J1-Pin_18-Pad18) -> /T527/PI0
- J1 pad 19: unconnected-(J1-Pin_19-Pad19) -> /T527/PI4
- J1 pad 2: unconnected-(J1-Pin_2-Pad2) -> 5V_SYS
- J1 pad 20: unconnected-(J1-Pin_20-Pad20) -> GND
- J1 pad 21: unconnected-(J1-Pin_21-Pad21) -> /T527/PI5
- J1 pad 22: unconnected-(J1-Pin_22-Pad22) -> /T527/PI1
- J1 pad 23: unconnected-(J1-Pin_23-Pad23) -> /T527/PI3
- J1 pad 24: unconnected-(J1-Pin_24-Pad24) -> /T527/PI2
- J1 pad 25: unconnected-(J1-Pin_25-Pad25) -> GND
- J1 pad 26: unconnected-(J1-Pin_26-Pad26) -> /T527/PI6
- J1 pad 27: unconnected-(J1-Pin_27-Pad27) -> /T527/PL9
- J1 pad 28: unconnected-(J1-Pin_28-Pad28) -> /T527/PL8
- J1 pad 29: unconnected-(J1-Pin_29-Pad29) -> /T527/PI9
- J1 pad 3: unconnected-(J1-Pin_3-Pad3) -> /T527/PL13
- J1 pad 30: unconnected-(J1-Pin_30-Pad30) -> GND
- J1 pad 31: unconnected-(J1-Pin_31-Pad31) -> /T527/PI10
- J1 pad 32: unconnected-(J1-Pin_32-Pad32) -> /T527/PI14
- J1 pad 33: unconnected-(J1-Pin_33-Pad33) -> /T527/PI11
- J1 pad 34: unconnected-(J1-Pin_34-Pad34) -> GND
- J1 pad 35: unconnected-(J1-Pin_35-Pad35) -> /T527/PI12
- J1 pad 36: unconnected-(J1-Pin_36-Pad36) -> /T527/PI15
- J1 pad 37: unconnected-(J1-Pin_37-Pad37) -> /T527/PI13
- J1 pad 38: unconnected-(J1-Pin_38-Pad38) -> /T527/PI8
- J1 pad 39: unconnected-(J1-Pin_39-Pad39) -> GND
- J1 pad 4: unconnected-(J1-Pin_4-Pad4) -> 5V_SYS
- J1 pad 40: unconnected-(J1-Pin_40-Pad40) -> /T527/PI7
- J1 pad 5: unconnected-(J1-Pin_5-Pad5) -> /T527/PL12
- J1 pad 6: unconnected-(J1-Pin_6-Pad6) -> GND
- J1 pad 7: unconnected-(J1-Pin_7-Pad7) -> /T527/PL11
- J1 pad 8: unconnected-(J1-Pin_8-Pad8) -> /T527/PL2
- J1 pad 9: unconnected-(J1-Pin_9-Pad9) -> GND
- R202 pad 1: GND -> VCC-3V3
- R202 pad 2: Net-(U17-A1_PRSNT#1) -> /T527/PCIE-CARD-PRESENT
- U17 pad 1: Net-(U17-A1_PRSNT#1) -> /T527/PCIE-CARD-PRESENT
- U8 pad AA7: unconnected-(U8F-GNDADC-PadAA7) -> AGND
- U8 pad AA9: unconnected-(U8A-VREFPADC-PadAA9) -> ALDO4
- U8 pad AB9: unconnected-(U8A-AVCC-PadAB9) -> ALDO4
- U8 pad AC7: unconnected-(U8A-VRP-PadAC7) -> /T527/VRP
- U8 pad AE3: unconnected-(U8F-AGND-PadAE3) -> AGND
- U8 pad AE7: unconnected-(U8A-ALDOOUT-PadAE7) -> ALDO-OUT
- U8 pad AG13: unconnected-(U8C-PI1-PadAG13) -> /T527/PI1
- U8 pad AG4: unconnected-(U8A-VRA2-PadAG4) -> /T527/VRA2
- U8 pad AG5: unconnected-(U8A-VRA1-PadAG5) -> /T527/VRA1
- U8 pad AH13: unconnected-(U8C-PI0-PadAH13) -> /T527/PI0
- U8 pad AH15: unconnected-(U8C-PI7-PadAH15) -> /T527/PI7
- U8 pad AH17: unconnected-(U8C-PI15-PadAH17) -> /T527/PI15
- U8 pad AJ11: unconnected-(U8A-RESET-PadAJ11) -> AP-RESET
- U8 pad AJ15: unconnected-(U8C-PI5-PadAJ15) -> /T527/PI5
- U8 pad AJ3: unconnected-(U8A-CPVDD-PadAJ3) -> CPVDD
- U8 pad AJ4: unconnected-(U8A-VEE-PadAJ4) -> Net-(U8A-CPVEE)
- U8 pad AJ5: unconnected-(U8A-CPVIN-PadAJ5) -> BLDO3
- U8 pad AJ7: unconnected-(U8C-PL13-PadAJ7) -> /T527/PL13
- U8 pad AJ9: unconnected-(U8C-PL11-PadAJ9) -> /T527/PL11
- U8 pad AK13: unconnected-(U8A-WREQIN-PadAK13) -> Net-(U8A-WREQIN)
- U8 pad AK15: unconnected-(U8C-PI6-PadAK15) -> /T527/PI6
- U8 pad AK17: unconnected-(U8C-PI13-PadAK17) -> /T527/PI13
- U8 pad AK2: unconnected-(U8A-CPVEE-PadAK2) -> Net-(U8A-CPVEE)
- U8 pad AK7: unconnected-(U8C-PL12-PadAK7) -> /T527/PL12
- U8 pad AK9: unconnected-(U8C-PL10-PadAK9) -> /T527/PL10
- U8 pad AL15: unconnected-(U8C-PI2-PadAL15) -> /T527/PI2
- U8 pad AL16: unconnected-(U8C-PI8-PadAL16) -> /T527/PI8
- U8 pad AL17: unconnected-(U8C-PI12-PadAL17) -> /T527/PI12
- U8 pad AL7: unconnected-(U8C-PL5-PadAL7) -> /T527/PL5
- U8 pad AM10: unconnected-(U8A-NMI-PadAM10) -> AP-NMI
- U8 pad AM15: unconnected-(U8C-PI4-PadAM15) -> /T527/PI4
- U8 pad AM16: unconnected-(U8C-PI9-PadAM16) -> /T527/PI9
- U8 pad AM17: unconnected-(U8C-PI11-PadAM17) -> /T527/PI11
- U8 pad AM18: unconnected-(U8C-PI14-PadAM18) -> /T527/PI14
- U8 pad AM6: unconnected-(U8C-PL3-PadAM6) -> /T527/PL3
- U8 pad AM7: unconnected-(U8C-PL4-PadAM7) -> /T527/PL4
- U8 pad AM8: unconnected-(U8C-PL7-PadAM8) -> /T527/PL7
- U8 pad AM9: unconnected-(U8C-PL9-PadAM9) -> /T527/PL9
- U8 pad AN15: unconnected-(U8C-PI3-PadAN15) -> /T527/PI3
- U8 pad AN17: unconnected-(U8C-PI10-PadAN17) -> /T527/PI10
- U8 pad AN2: /T527/BT-WAKE-AP -> /T527/AP-WAKE-BT
- U8 pad AN3: /T527/AP-WAKE-BT -> /T527/BT-WAKE-AP
- U8 pad AN7: unconnected-(U8C-PL2-PadAN7) -> /T527/PL2
- U8 pad AN8: unconnected-(U8C-PL6-PadAN8) -> /T527/PL6
- U8 pad AN9: unconnected-(U8C-PL8-PadAN9) -> /T527/PL8
- U8 pad F16: unconnected-(U8A-FEL-PadF16) -> /T527/FEL
- U8 pad L28: unconnected-(U8D-PD20-PadL28) -> /T527/PCIE-CARD-PRESENT
- U8 pad L29: unconnected-(U8D-PD21-PadL29) -> /T527/PCIE-SEL
- U8 pad Y10: unconnected-(U8A-VREFNADC-PadY10) -> AGND
- U8 pad Y9: unconnected-(U8A-VCMADC-PadY9) -> VCM-ADC
Routing:
- net /T527/PI11: track 0.00 -> 49.3 mm, vias 0 -> 1
- net /T527/PI7: track 0.00 -> 48.0 mm, vias 0 -> 1
- net /T527/PI15: track 0.00 -> 47.7 mm, vias 0 -> 1
- net /T527/PI8: track 0.00 -> 44.4 mm, vias 0 -> 1
- net /T527/PI13: track 0.00 -> 44.3 mm, vias 0 -> 1
- net /T527/PI2: track 0.00 -> 42.6 mm, vias 0 -> 1
- net /T527/PI12: track 0.00 -> 40.2 mm, vias 0 -> 1
- net /T527/PCIE-CARD-PRESENT: track 0.00 -> 35.4 mm, vias 0 -> 2
- net /T527/PI10: track 0.00 -> 35.3 mm, vias 0 -> 1
- net /T527/PI6: track 0.00 -> 33.9 mm, vias 0 -> 1
- net /T527/PI9: track 0.00 -> 33.0 mm, vias 0 -> 1
- net /T527/PL13: track 0.00 -> 32.9 mm, vias 0 -> 1
- net /T527/PI1: track 0.00 -> 32.0 mm, vias 0 -> 1
- net /T527/PI5: track 0.00 -> 30.9 mm, vias 0 -> 1
- net /T527/PL12: track 0.00 -> 30.9 mm, vias 0 -> 1
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Other:
- board text added: "BOOT 1"
- board text added: "RESET"

Commit message: revert back to this version if reroute fails
Parts:
- added G***: LOGO, LOGO, F.Cu at (130.0, 80.8)
- R207, R208, R209, R210, R211, R212: moved to F.Cu
- moved R184 9.88 mm to (145.0, 126.0), turned to 0 degrees
- moved C376 8.47 mm to (95.6, 103.1), turned to 0 degrees
- moved D3 6.91 mm to (146.4, 123.5)
- moved Q3 6.38 mm to (144.4, 128.4), turned to -90 degrees
- moved C389 5.92 mm to (106.8, 105.9)
- moved R185 2.72 mm to (144.7, 130.8), turned to 180 degrees
- moved R182 2.02 mm to (141.3, 130.8), turned to 0 degrees
- moved C382 1.70 mm to (94.6, 103.8)
- moved R212 1.24 mm to (84.8, 107.2)
- moved R210 1.24 mm to (84.8, 105.7)
- moved C9 1.00 mm to (149.1, 128.2)
- moved R159 1.00 mm to (150.9, 128.2)
- moved C195 0.92 mm to (143.4, 125.9), turned to 180 degrees
- moved C292 0.81 mm to (149.0, 101.5)
- moved C293 0.81 mm to (147.6, 101.5)
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Routing:
- net 5V_SYS: track 0.00 -> 22.4 mm, vias 0 -> 2
- net DCDC2: track 0.00 -> 15.5 mm, vias 0 -> 17
- net /power input/CC1: track 0.50 -> 12.1 mm
- net +12V: track 0.00 -> 11.0 mm
- net AUX-3V3: track 0.00 -> 10.9 mm
- net /power input/CC2: track 0.50 -> 10.7 mm
- net /power input/VBUS_MAIN: track 13.8 -> 23.4 mm
- net /power input/V_MAIN: track 1.27 -> 9.14 mm
- net /power input/POWER_OK3: track 0.00 -> 7.48 mm, vias 0 -> 2
- net BLDO3: track 0.00 -> 6.63 mm, vias 0 -> 7
- net 323-DCDC1/2: track 0.00 -> 6.49 mm, vias 0 -> 5
- net Net-(Q1-S-Pad1): track 0.00 -> 6.37 mm
- net DCDC4: track 0.00 -> 6.14 mm, vias 0 -> 7
- net ALDO4: track 0.00 -> 5.75 mm, vias 0 -> 5
- net Net-(U6-SW): track 0.00 -> 5.60 mm
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Other:
- board text added: "ETH 0"
- board text added: "ETH 1"
- board text added: "LPDDR4X"
- board text added: "PCIe"
- board text added: "T527"
- board text added: "USB 2.0"
- board text added: "USB 3.0"
