File: PCB/Artificer A1 Board Rev 0.1/Artificer A1 Board Rev 0.1.kicad_pcb (KiCad board)
At the start: 6 copper layers, 115 x 90 mm, 507 parts, among them CN1 PJ-327A0-SMT, J1 Conn_02x20_Odd_Even, J2 Conn_01x02, M1 Fan&Heatsink_40x40mm, Q1 AON3419-TP, Q2 AON3419-TP, Q3 AO3401A, Q4 2SK3018, Q6 AO3401A, Q7 AO3401A, SW1 BOOT1, SW2 RESET, U1 GT-USB-7010ASV, U10 AXP717B, U11 AXP323, U12 K4UBE3D4AB-MGCL, U13 AFC11-S22ICA-00, U14 RTL8211F-CG, U15 RTL8211F-CG, U16 HD3SS3202IRSVR, U17 X3113WVS-36-9TV01, U2 GD25LQ128EWIGR, U21 CH217K, U22 CH334F_C5187527, U24 AFC11-S22ICA-00, U25 AFC11-S22ICA-00, U26 AFC11-S22ICA-00, U3 AP64500SP-13, U4 STUSB4500QTR, U5 AP64350SP-13, U6 AP64500SP-13, U8 T527M00X0DCH, U9 SY8089A1AAC, X1 25MHz, X2 25MHz, X3 SMD-3225_4P12M12PF10PPM, X4 25MHz, X5 SC-20S32.768kHz20PPM9pF

Commit message: now the board is more manufacturable
Parts:
- C168, C210, R200, R201: moved to B.Cu
- moved C282 61.3 mm to (35.5, 91.9)
- moved C326 61.3 mm to (40.2, 94.8)
- moved C329 61.3 mm to (36.0, 96.8)
- moved C331 61.3 mm to (35.2, 96.8)
- moved C337 61.3 mm to (28.7, 95.0)
- moved C340 61.3 mm to (28.6, 96.8)
- moved C342 61.3 mm to (38.2, 97.5)
- moved C343 61.3 mm to (38.9, 97.5)
- moved C348 61.3 mm to (34.1, 92.0)
- moved C349 61.3 mm to (38.5, 89.6)
- moved C350 61.3 mm to (34.4, 90.9)
- moved C352 61.3 mm to (32.8, 88.6)
- moved C356 61.3 mm to (37.1, 91.1)
- moved C357 61.3 mm to (37.0, 89.6)
- moved C358 61.3 mm to (35.5, 90.4)
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Connections:
- net Net-(U8D-PCIEREFCLKN) renamed /T527/PCIE-CLKN
- net Net-(U8D-PCIEREFCLKP) renamed /T527/PCIE-CLKP
- net Net-(U8D-PCIETX0-DN/USB) renamed /T527/PCIE-DN
- net Net-(U8D-PCIETX0-DP/USB) renamed /T527/PCIE-DP
Routing:
- net /T527/FEL: track 0.00 -> 64.7 mm, vias 0 -> 2
- net GND: track 14.0 -> 64.0 mm, vias 128 -> 71
- net /T527/PI11: track 49.3 -> 0.00 mm, vias 1 -> 0
- net /T527/PI7: track 48.0 -> 0.50 mm
- net /T527/PI15: track 47.7 -> 0.50 mm
- net /T527/PI8: track 44.4 -> 0.00 mm, vias 1 -> 0
- net /T527/AP-WAKE-BT: track 44.0 -> 0.00 mm, vias 2 -> 0
- net /T527/PI13: track 44.3 -> 0.50 mm
- net /T527/PI2: track 42.6 -> 0.00 mm, vias 1 -> 0
- net /T527/BT-WAKE-AP: track 41.2 -> 0.00 mm, vias 2 -> 0
- net /T527/PWR-EN: track 40.5 -> 0.00 mm, vias 2 -> 0
- net /T527/PI12: track 40.2 -> 0.00 mm, vias 1 -> 0
- net /T527/WL-WAKE-AP: track 38.2 -> 0.00 mm, vias 2 -> 0
- net /T527/PCIE-CARD-PRESENT: track 35.4 -> 0.00 mm, vias 2 -> 0
- net /T527/PI10: track 35.3 -> 0.00 mm, vias 1 -> 0
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
Commit message: finished ddr4 and gpio
Parts:
- R178, R179: moved to B.Cu
- moved C305 2.49 mm to (93.3, 114.8)
- moved C304 2.49 mm to (95.0, 114.8)
- moved X4 2.49 mm to (94.1, 117.0)
- moved X5 1.92 mm to (89.8, 116.7)
- moved C306 1.92 mm to (90.5, 118.1)
- moved R206 1.92 mm to (89.8, 115.3)
- moved C307 1.92 mm to (89.1, 118.1)
- moved R179 0.50 mm to (113.3, 120.3)
- moved R178 0.38 mm to (113.3, 118.3)
- moved C319 0.10 mm to (110.2, 118.8)
- moved C325 0.10 mm to (110.2, 119.7)
Connections:
- J1 pad 11: /T527/PL4 -> /T527/PL6
- J1 pad 15: /T527/PL6 -> /T527/PL11
- J1 pad 16: /T527/PL7 -> unconnected-(J1-Pin_16-Pad16)
- J1 pad 27: /T527/PL9 -> /T527/PL13
- J1 pad 28: /T527/PL8 -> /T527/PL12
- J1 pad 3: /T527/PL13 -> /T527/PL9
- J1 pad 5: /T527/PL12 -> /T527/PL8
- J1 pad 7: /T527/PL11 -> /T527/PL7
- U8 pad AM7: /T527/PL4 -> GND
Routing:
- net /T527/HP-DET: track 0.00 -> 105.2 mm, vias 0 -> 1
- net Net-(U8A-MICDET): track 0.00 -> 103.5 mm, vias 0 -> 1
- net /T527/HBIAS: track 0.00 -> 103.1 mm, vias 0 -> 1
- net /T527/HPOUTL: track 0.00 -> 102.5 mm, vias 0 -> 1
- net /T527/HPOUTFB: track 0.00 -> 100.4 mm, vias 0 -> 1
- net /T527/HPOUTR: track 0.00 -> 99.8 mm, vias 0 -> 2
- net AP-NMI: track 0.00 -> 74.6 mm, vias 0 -> 2
- net /T527/PMU-SDA: track 0.00 -> 61.6 mm, vias 0 -> 2
- net /T527/PMU-SCK: track 0.00 -> 58.2 mm, vias 0 -> 2
- net /T527/PI15: track 0.50 -> 57.7 mm
- net /T527/PI12: track 0.00 -> 56.3 mm, vias 0 -> 1
- net /T527/PI7: track 0.50 -> 51.4 mm
- net /T527/PI8: track 0.00 -> 50.5 mm, vias 0 -> 1
- net /T527/PI13: track 0.50 -> 48.8 mm
- net GND: track 64.0 -> 110.6 mm, vias 71 -> 132
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- removed copper zone on F.Cu, net /power input/V_MAIN
Other:
- board text removed: "LPDDR4X"

Commit message: finished bga decoupling placement
Parts:
- R154: moved to F.Cu
- moved C327 76.4 mm to (111.8, 105.3), turned to 180 degrees
- moved C326 72.2 mm to (111.9, 103.2)
- moved C382 63.9 mm to (97.4, 103.0), turned to 180 degrees
- moved C350 63.2 mm to (97.0, 100.0)
- moved C391 63.1 mm to (94.5, 101.1), turned to 180 degrees
- moved C357 62.9 mm to (98.8, 101.3), turned to 180 degrees
- moved C383 62.9 mm to (97.4, 103.8), turned to 180 degrees
- moved C392 62.5 mm to (94.5, 101.8), turned to 180 degrees
- moved C397 62.4 mm to (92.7, 101.6), turned to 180 degrees
- moved C423 62.3 mm to (100.3, 101.3)
- moved C348 62.3 mm to (95.9, 99.5)
- moved C412 62.1 mm to (100.0, 100.3)
- moved C409 62.0 mm to (99.8, 98.2), turned to -90 degrees
- moved C358 62.0 mm to (97.0, 98.5), turned to -90 degrees
- moved C420 61.9 mm to (92.8, 98.2), turned to -90 degrees
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Routing:
- net Net-(U8A-MICDET): track 103.5 -> 3.50 mm, vias 1 -> 0
- net /T527/HS-MIC: track 0.00 -> 99.5 mm, vias 0 -> 1
- net GND: track 110.6 -> 182.2 mm, vias 132 -> 177
- net /T527/PCIE-CARD-PRESENT: track 0.00 -> 36.3 mm, vias 0 -> 2
- net /T527/PCIE-SEL: track 0.50 -> 23.4 mm, vias 1 -> 2
- net DCDC2: track 0.00 -> 10.0 mm, vias 0 -> 8
- net Net-(JP1-SIG): track 0.00 -> 8.81 mm
- net 323-DCDC1/2: track 0.00 -> 4.50 mm, vias 0 -> 2
- net DCDC3: track 13.3 -> 17.8 mm, vias 26 -> 29
- net DCDC4: track 0.00 -> 4.41 mm, vias 0 -> 6
- net /wifi&bt/ANT0: track 0.00 -> 3.93 mm
- net DCDC1: track 0.00 -> 3.71 mm, vias 0 -> 2
- net VDD06-DRAM: track 9.77 -> 13.3 mm, vias 20 -> 22
- net 323-DCDC3: track 0.00 -> 2.50 mm, vias 0 -> 2
- net AGND: track 0.50 -> 2.75 mm, vias 1 -> 2
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