File: PCB/Artificer A1 Board Rev 0.1/Artificer A1 Board Rev 0.1.kicad_pcb (KiCad board)
At the start: 6 copper layers, 115 x 90 mm, 507 parts, among them CN3 PJ-393-8P_C49284725, J1 Conn_02x20_Odd_Even, J2 Conn_01x02, M1 Fan&Heatsink_40x40mm, Q1 AON3419-TP, Q2 AON3419-TP, Q3 AO3401A, Q4 2SK3018, Q6 AO3401A, Q7 AO3401A, SW1 BOOT1, SW2 RESET, U1 GT-USB-7010ASV, U10 AXP717B, U11 AXP323, U12 K4UBE3D4AB-MGCL, U13 AFC11-S22ICA-00, U14 RTL8211F-CG, U15 RTL8211F-CG, U16 HD3SS3202IRSVR, U17 X3113WVS-36-9TV01, U2 GD25LQ128EWIGR, U21 CH217K, U22 CH334F_C5187527, U24 AFC11-S22ICA-00, U25 AFC11-S22ICA-00, U26 AFC11-S22ICA-00, U3 AP64500SP-13, U4 STUSB4500QTR, U5 AP64350SP-13, U6 AP64500SP-13, U8 T527M00X0DCH, U9 SY8089A1AAC, X1 25MHz, X2 25MHz, X3 SMD-3225_4P12M12PF10PPM, X4 25MHz, X5 SC-20S32.768kHz20PPM9pF

Commit message: 3.3V Aux & 12V power
Parts:
- moved C15 4.71 mm to (139.0, 116.1), turned to 90 degrees
- moved C294 4.08 mm to (149.4, 99.2), turned to 180 degrees
- moved C293 2.03 mm to (149.4, 100.7), turned to 180 degrees
- moved C292 0.78 mm to (149.4, 102.2), turned to 180 degrees
- moved C176 0.71 mm to (99.8, 82.5)
Routing:
- net CPUSLDO: track 2.07 -> 72.5 mm
- net /T527/PI1: track 0.50 -> 33.8 mm, vias 1 -> 2
- net Net-(R146-Pad1): track 0.00 -> 31.4 mm, vias 0 -> 1
- net Net-(R144-Pad1): track 0.00 -> 30.5 mm, vias 0 -> 1
- net /T527/PI5: track 5.94 -> 29.5 mm
- net /ETH0.RGMII-RXCTL: track 51.6 -> 29.3 mm
- net /ETH0.RGMII-RXD0: track 52.5 -> 30.3 mm
- net +12V: track 19.0 -> 0.00 mm, vias 0 -> 32
- net /T527/PCIE0-PERSTN: track 18.4 -> 34.3 mm, vias 1 -> 2
- net /ETH0.RGMII-CLKIN: track 30.8 -> 43.7 mm
- net 5V_SYS: track 25.9 -> 16.7 mm, vias 12 -> 20
- net DCDC4: track 14.0 -> 20.9 mm, vias 44 -> 59
- net /T527/PCIE0-CLKREQN: track 52.4 -> 58.7 mm
- net /ETH0.RGMII-PHYRSTB: track 41.4 -> 36.6 mm
- net AUX-3V3: track 5.79 -> 1.21 mm, vias 0 -> 16
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- added copper zone on F.Cu, net +12V
- added copper zone on In2.Cu, net +12V
- added copper zone on In2.Cu, net 5V_SYS
- added copper zone on B.Cu, net AUX-3V3
- added copper zone on F.Cu, net AUX-3V3
- added copper zone on In3.Cu, net PS

Commit message: getting closer
Parts:
- removed C349: 2.2uF, Capacitor_SMD:C_0201_0603Metric
- removed C357: 100nF, Capacitor_SMD:C_0201_0603Metric
- moved C252 3.20 mm to (132.2, 115.2), turned to 90 degrees
- moved C266 2.14 mm to (144.7, 61.8)
- moved C265 2.14 mm to (146.2, 61.8)
- moved R110 1.98 mm to (153.2, 68.9), turned to 0 degrees
- moved C212 1.00 mm to (58.8, 76.5)
- moved C214 1.00 mm to (58.8, 75.8)
- moved C189 0.85 mm to (57.8, 121.7)
- moved C190 0.85 mm to (57.8, 122.5)
- moved C193 0.78 mm to (57.9, 95.5)
- moved C194 0.78 mm to (57.9, 96.3)
- moved C387 0.72 mm to (114.5, 103.2)
- moved C389 0.72 mm to (116.0, 103.2)
- moved C385 0.72 mm to (111.5, 103.2)
- moved C394 0.72 mm to (113.0, 103.2)
- moved C412 0.67 mm to (99.3, 100.3)
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Routing:
- net DCDC4: track 20.9 -> 178.5 mm, vias 59 -> 61
- net AP-RESET: track 19.9 -> 166.0 mm, vias 2 -> 4
- net /T527/DBG_UART0_RX: track 46.0 -> 102.7 mm, vias 3 -> 4
- net /T527/DBG_UART0_TX: track 47.2 -> 101.8 mm, vias 2 -> 3
- net 5V_SYS: track 16.7 -> 56.2 mm, vias 20 -> 35
- net VBUS_USB2.0: track 0.00 -> 35.7 mm
- net BLDO2: track 70.2 -> 80.9 mm, vias 9 -> 11
- net GND: track 261.0 -> 271.5 mm, vias 238 -> 273
- net VDD06-DRAM: track 87.1 -> 93.7 mm
- net ALDO4: track 106.2 -> 111.9 mm
- net BLDO1: track 109.5 -> 114.7 mm
- net /ethernet0/GM_VDD10: track 0.00 -> 3.83 mm, vias 0 -> 6
- net /ETH1.RGMII-RXD2: track 41.9 -> 45.7 mm
- net /ethernet 1/GM_VDD10: track 0.00 -> 3.56 mm, vias 0 -> 5
- net /T527/HSCL: track 84.6 -> 81.6 mm
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