File: PCB/Artificer A1 Board Rev 0.1/T527 power.kicad_sch (KiCad schematic)
At the start: 1 part, among them U8 T527M00X0DCH

Commit message: more routing and decoupling
Parts:
- added C282, C285, C286, C328, C329, C330, C331, C341, C342, C348, C349, C350, C351, C352, C379, C380, C381, C386, C388, C390, C391, C395, C396, C397, C400, C401, C402, C404, C405, C425: 2.2uF, Capacitor_SMD:C_0201_0603Metric, symbol Cap:JLCPCB_Lib_Blank_Cap
- added C283, C284, C377, C378, C385, C387, C389, C394, C399: 22uF, Capacitor_SMD:C_0603_1608Metric, symbol Cap:JLCPCB_Lib_Blank_Cap
- added C326, C327: 10uF, Capacitor_SMD:C_0402_1005Metric, symbol Cap:JLCPCB_Lib_Blank_Cap
- added C343, C344, C345, C346, C347, C356, C357, C358, C359, C360, C363, C364, C365, C375, C376, C383, C384, C392, C393, C398, C403, C406, C408, C410, C411, C412, C413, C414, C415, C416, C418, C419, C420, C421, C422, C423, C424, C426, C427, C428: 100nF, Capacitor_SMD:C_0201_0603Metric, symbol Cap:JLCPCB_Lib_Blank_Cap
- added C374, C382, C407, C409, C417: 1uF, Capacitor_SMD:C_0201_0603Metric, symbol Cap:JLCPCB_Lib_Blank_Cap
Connections:
- net GND: now also C282.1, C283.1, C284.1, C285.1, C286.1, C326.1, C327.1, C328.1, C329.1, C330.1, C331.1, C341.1, C342.1, C343.1, C344.1, C345.1, C346.1, C347.1, C348.1, C349.1, C350.1, C351.1, C352.1, C356.1, C357.1, C358.1, C359.1, C360.1, C363.1, C364.1, C365.1, C374.1, C375.1, C376.1, C377.1, C378.1, C379.1, C380.1, C381.1, C382.1, C383.1, C384.1, C385.1, C386.1, C387.1, C388.1, C389.1, C390.1, C391.1, C392.1, C393.1, C394.1, C395.1, C396.1, C397.1, C398.1, C399.1, C400.1, C401.1, C402.1, C403.1, C404.1, C405.1, C406.1, C407.1, C408.1, C409.1, C410.1, C411.1, C412.1, C413.1, C414.1, C415.1, C416.1, C417.1, C418.1, C419.1, C420.1, C421.1, C422.1, C423.1, C424.1, C425.1, C426.1, C427.1, C428.1
- net VCC-DCXO: now also C426.2
- net VCC-EFUSE: now also C423.2
- net VCC-IO: now also C407.2, C408.2
- net VCC-LVDS0: now also C412.2
- net VCC-LVDS1: now also C413.2
- net VCC-MCSI: now also C420.2
- net VCC-PC: now also C410.2
- net VCC-PD: now also C409.2, C411.2
- net VCC-PE: now also C414.2
- net VCC-PG: now also C415.2
- net VCC-PI: now also C416.2
- net VCC-PJ: now also C417.2, C418.2
- net VCC-PK: now also C419.2
- net VCC-PL: now also C421.2
- net VCC-PLL: now also C425.2
- net VCC-PM: now also C422.2
- net VCC-RTC: now also C424.2
- net VCC18-EDP: now also C341.2, C356.2
- net VCC18-HDMI: now also C349.2, C357.2
- net VCC18-PCIE: now also C351.2, C359.2
- net VCC33-USB: now also C363.2
- net VCC33-USB-2: now also C365.2
- net VDD-CPUB: now also C282.2, C283.2, C284.2, C285.2, C286.2, C374.2, C375.2, C376.2
- net VDD-CPUL: now also C377.2, C378.2, C379.2, C380.2, C381.2, C382.2, C383.2, C384.2
- net VDD-CPUS: now also C405.2, C406.2
- net VDD-DE: now also C385.2, C386.2
- net VDD-DNR: now also C399.2, C400.2, C401.2, C402.2, C403.2, C404.2
- net VDD-GPU: now also C394.2, C395.2, C396.2, C397.2, C398.2
- net VDD-SYS: now also C389.2, C390.2, C391.2, C392.2, C393.2
- net VDD-VE: now also C387.2, C388.2
- net VDD09-EDP: now also C348.2, C427.2
- net VDD09-HDMI: now also C350.2, C358.2
- net VDD09-PCIE: now also C352.2, C360.2
- net VDD09-USB: now also C364.2
- net VDD33: now also C428.2
- net AGND: now reaches U8.AA7 (GNDADC)
- net AGND: now also U8.AE3 (AGND)
- new net VDD06-DRAM: C327.2, C329.2, C331.2, C346.2, C347.2
- new net VDD11-DRAM: C326.2, C328.2, C330.2, C344.2, C345.2
- new net VDD18-DRAM: C342.2, C343.2
Other:
- note added: "Memory Controller"
- note removed: "CPVEE, CPVDD, These pins are used for headphones and negative charge pumps. Probably shouldnt be here"
- moved on the sheet: U8B

Commit message: added power and gnd vias
Parts:
- C343, C349, C357: now not fitted; now left out of the parts list
Changed lines of the file:
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@@
 		(body_style 1)
 		(exclude_from_sim no)
-		(in_bom yes)
-		(on_board yes)
-		(in_pos_files yes)
-		(dnp no)
+		(in_bom no)
+		(on_board no)
+		(in_pos_files no)
+		(dnp yes)
 		(property "Reference" "C343"
 			(at 114.808 210.82 0)
@@
 		(body_style 1)
 		(exclude_from_sim no)
-		(in_bom yes)
-		(on_board yes)
-		(in_pos_files yes)
-		(dnp no)
+		(in_bom no)
+		(on_board no)
+		(in_pos_files no)
+		(dnp yes)
 		(property "Reference" "C349"
 			(at 330.708 101.6 0)
@@
 		(body_style 1)
 		(exclude_from_sim no)
-		(in_bom yes)
-		(on_board yes)
-		(in_pos_files yes)
-		(dnp no)
+		(in_bom no)
+		(on_board no)
+		(in_pos_files no)
+		(dnp yes)
 		(property "Reference" "C357"
 			(at 339.598 101.6 0)
